File: Electronic Design/Interactive Core Memory Badge v0.1/Interactive Core Memory Badge v0.1.kicad_pcb (KiCad board)
At the start: 2 copper layers, 81.3 x 165.1 mm, 101 parts, among them M1 LED_Array, M2 OLED_DISPLAY, Q1 MMBT4403LT1G, Q10 MMBT4401LT1G, Q11 MMBT4403LT1G, Q12 MMBT4401LT1G, Q13 MMBT4403LT1G, Q14 MMBT4401LT1G, Q15 MMBT4403LT1G, Q16 MMBT4401LT1G, Q17 MMBT4403LT1G, Q18 MMBT4401LT1G, Q19 MMBT4403LT1G, Q2 MMBT4401LT1G, Q20 MMBT4401LT1G, Q21 MMBT4401LT1G, Q3 MMBT4403LT1G, Q4 MMBT4401LT1G, Q5 MMBT4403LT1G, Q6 MMBT4401LT1G, Q7 MMBT4403LT1G, Q8 MMBT4401LT1G, Q9 MMBT4403LT1G, SW1 SW_SPST, SW2 SW_Reed, U1 Micro_LiPo_Charger, U2 Teensy-LC, U3 LM393, U4 A3214ELHLT-T

Commit message: Prototype release V0.1
Parts:
- removed M1: LED_Array, Core_Memory_8x8_Array:LED_Matrix_Header_3pin
- removed M2: OLED_DISPLAY, Core_Memory_8x8_Array:OLED_Header_4PIN
- added D10: BAT54CW, Package_TO_SOT_SMD:SOT-323_SC-70, F.Cu at (63.5, 54.6)
- added D11: BAT54AW, Package_TO_SOT_SMD:SOT-323_SC-70, F.Cu at (63.5, 61.0)
- added D12: BAT54CW, Package_TO_SOT_SMD:SOT-323_SC-70, F.Cu at (63.5, 67.9)
- added D7: BAT54AW, Package_TO_SOT_SMD:SOT-323_SC-70, F.Cu at (71.1, 109.9)
- added D8: BAT54CW, Package_TO_SOT_SMD:SOT-323_SC-70, F.Cu at (78.1, 109.9)
- added D9: BAT54AW, Package_TO_SOT_SMD:SOT-323_SC-70, F.Cu at (63.5, 47.6)
- added H1: LED_Array, Core_Memory_8x8_Array:LED_Matrix_Header_3pin, F.Cu at (75.6, 115.6)
- added H2: OLED_DISPLAY, Core_Memory_8x8_Array:OLED_Header_4PIN, F.Cu at (98.4, 138.4)
- D1, D3, D5: value BAW56S -> BAT54AW; footprint Package_TO_SOT_SMD:SOT-363_SC-70-6 -> Package_TO_SOT_SMD:SOT-323_SC-70
- D2, D4, D6: value BAV70S -> BAT54CW; footprint Package_TO_SOT_SMD:SOT-363_SC-70-6 -> Package_TO_SOT_SMD:SOT-323_SC-70
- moved D5 118.1 mm to (91.4, 109.9)
- moved Q19 106.2 mm to (61.6, 120.7), turned to 180 degrees
- moved D6 105.6 mm to (85.1, 109.9), turned to 180 degrees
- moved Q17 77.3 mm to (61.6, 133.3), turned to 180 degrees
- moved R30 73.3 mm to (107.3, 144.8)
- moved D3 73.3 mm to (104.8, 109.9)
- moved R34 71.1 mm to (122.6, 144.8)
- moved D1 68.6 mm to (111.1, 109.9), turned to 180 degrees
- moved Q10 68.6 mm to (68.6, 122.6), turned to 180 degrees
- moved R11 68.4 mm to (63.5, 101.6), turned to 270 degrees
- moved R33 67.8 mm to (115.6, 144.8)
- moved R35 67.4 mm to (122.6, 140.3), turned to 0 degrees
- moved R12 67.1 mm to (66.0, 101.6), turned to 270 degrees
- moved C1 66.9 mm to (64.1, 40.6), turned to 180 degrees
- moved R32 65.2 mm to (122.6, 135.9)
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Connections:
- D1 pad 1: XB0 -> XB1
- D1 pad 2: XB1 -> XB0
- D3 pad 1: XB4 -> XB3
- D3 pad 2: XB5 -> XB2
- D3 pad 3: Net-(D3-Pad3) -> Net-(D1-Pad3)
- D4 pad 1: XB4 -> XB2
- D4 pad 2: XB5 -> XB3
- D4 pad 3: Net-(D4-Pad3) -> Net-(D2-Pad3)
- D5 pad 1: YL1 -> XB5
- D5 pad 2: YL3 -> XB4
- D6 pad 1: YL0 -> XB4
- D6 pad 2: YL1 -> XB5
- Q17 pad 3: Net-(D5-Pad3) -> Net-(D9-Pad3)
- Q18 pad 3: Net-(D6-Pad6) -> Net-(D10-Pad3)
- Q19 pad 3: Net-(D5-Pad3) -> Net-(D11-Pad3)
- Q20 pad 3: Net-(D6-Pad3) -> Net-(D12-Pad3)
- Q5 pad 3: Net-(D3-Pad3) -> Net-(D5-Pad3)
- Q6 pad 3: Net-(D4-Pad3) -> Net-(D6-Pad3)
Routing:
- net Net-(D5-Pad3): track 0.00 -> 131.0 mm, vias 0 -> 2
- net Net-(D6-Pad3): track 0.00 -> 104.4 mm, vias 0 -> 2
- net SENSE_PULSE: track 0.00 -> 102.2 mm, vias 0 -> 4
- net Net-(D9-Pad3): track 0.00 -> 95.7 mm, vias 0 -> 2
- net +VSW: track 208.4 -> 296.2 mm, vias 11 -> 17
- net Net-(D10-Pad3): track 0.00 -> 79.9 mm, vias 0 -> 2
- net Net-(D11-Pad3): track 0.00 -> 64.6 mm, vias 0 -> 2
- net Net-(D2-Pad3): track 57.6 -> 118.0 mm, vias 1 -> 2
- net +3V3: track 332.2 -> 386.8 mm
- net Net-(D4-Pad3): track 53.6 -> 0.00 mm, vias 1 -> 0
- net Net-(D3-Pad3): track 53.1 -> 0.00 mm, vias 1 -> 0
- net SENSE1: track 19.7 -> 72.0 mm, vias 0 -> 2
- net Net-(D12-Pad3): track 0.00 -> 48.6 mm, vias 0 -> 2
- net Net-(Q11-Pad1): track 28.5 -> 77.1 mm, vias 1 -> 2
- net Net-(Q9-Pad1): track 26.6 -> 74.8 mm, vias 1 -> 2
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Other:
- outline, holes or cut-outs redrawn
- board text added: "Andy Geppert 2019"
- board text added: "CORE 64"
- board text added: "CORE 64 VERSION 0.1 INTERACTIVE CORE MEMORY BADGE"
- board text added: "Interactive Core Memory"
- board text added: "Micro LiPo Charger"
- board text added: "Power Switch"
- board text added: "Q10N"
- board text added: "Q10P"
- board text added: "Q2N"
- board text added: "Q2P"
- board text added: "Q3N"
- board text added: "Q3P"
- board text added: "Q4N"
- board text added: "Q4P"
- board text added: "Q5N"
- board text added: "Q5P"
- board text added: "Q6N"
- board text added: "Q6P"
- board text added: "Q7N"
- board text added: "Q7P"
- board text added: "Q8N"
- board text added: "Q8P"
- board text added: "Q9N"
- board text added: "Q9P"
- board text added: "Teensy LC"
- board text added: "WWW.MACHINEIDEAS.COM 2019 ANDY GEPPERT"
- board text added: "www.MachineIdeas.com"
- board text removed: "CORE 64 V0.1 INTERACTIVE CORE MEMORY BADGE"
- board text removed: "MACHINE IDEAS, LLC ANDY GEPPERT - 2019"
