File: Electronic Design/Interactive Core Memory Badge v0.2/Interactive Core Memory Badge v0.2.kicad_pcb (KiCad board)
At the start: 2 copper layers, 81.3 x 165.1 mm, 122 parts, among them Q1 MMBT4403LT1G, Q10 MMBT4401LT1G, Q11 MMBT4403LT1G, Q12 MMBT4401LT1G, Q13 MMBT4403LT1G, Q14 MMBT4401LT1G, Q15 MMBT4403LT1G, Q16 MMBT4401LT1G, Q17 MMBT4403LT1G, Q18 MMBT4401LT1G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

Commit message: Clean-up V0.2 PCB
Parts:
- moved TP12 0.64 mm to (114.3, 118.7)
Routing:
- net +3V3: track 407.0 -> 406.1 mm
Other:
- board text added: "CORE 64 VERSION 0.2 INTERACTIVE CORE MEMORY BADGE"
- board text removed: "CORE 64 VERSION 0.1 INTERACTIVE CORE MEMORY BADGE"

Commit message: Tweaks to V0.2 schematic and layout from notes.
Other:
- board text added: "CURRENT SENSE"
Changed lines of the file:
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@@
   (general
     (thickness 1.6)
-    (drawings 70)
+    (drawings 71)
     (tracks 1022)
     (zones 0)
@@
     (pad 6 smd rect (at 2.5 -2.75 270) (size 1.2 2.5) (layers F.Cu F.Paste F.Mask))
   )
+  (gr_text "CURRENT\nSENSE" (at 58.42 139.065) (layer F.SilkS)
+    (effects (font (size 1 1) (thickness 0.15)))
+  )
   (gr_text "Power\nSwitch" (at 58.42 152.4) (layer F.SilkS)

Commit message: Update v0.2 with correct Pimoroni footprint
Parts:
- CM1: footprint Core_Memory_8x8_Array:core_64 -> Core_Memory_8x8_Array:core_64_x6.7_y6.5mm
- R43: value 0 -> 0.01
- moved D1 0.25 mm to (111.4, 109.9)
- moved D8 0.15 mm to (78.0, 109.9)
- moved D3 0.10 mm to (104.7, 109.9)
Routing:
- net XT2-6: track 158.3 -> 160.3 mm
- net XT1-5: track 144.5 -> 142.9 mm
- net XT0-4: track 130.6 -> 132.0 mm
- net XT3-7: track 171.9 -> 172.9 mm
- net SENSE1: track 72.5 -> 73.3 mm
- net Net-(CM1-Pad27): track 27.4 -> 28.1 mm
- net Net-(D5-Pad3): track 131.0 -> 131.8 mm
- net YL1: track 16.3 -> 16.9 mm
