File: Electronic Design/Interactive Core Memory Badge (Logic) v0.3/Interactive Core Memory Badge (Logic) MCU v0.3.sch (KiCad schematic (older format))
At the start: 48 parts, among them Q22 MMBT4401LT1G, Q23 MMBT4401LT1G, SW2 SW_Reed, U2 Teensy-LC, U3 LM393, U5 A3214ELHLT-T

Commit message: Split V0.3 into two project boards
Parts:
- removed C5: 0.1uF, Capacitor_SMD:C_0805_2012Metric, symbol Device:CP1_Small
- removed C7: 10pF, Capacitor_SMD:C_0805_2012Metric, symbol Device:CP1_Small
- removed H2: LED_Array, Core_Memory_8x8_Array:LED_Matrix_Header_3pin, symbol Motor:Fan_3pin
- removed R47, R48: 4K7, Resistor_SMD:R_0805_2012Metric, symbol Device:R
- removed SW2: SW_Reed, Button_Switch_SMD:SW_SPST_REED_CT10-XXXX-G1, symbol Switch:SW_Reed
- removed TP20: REED_SWITCH, TestPoint:TestPoint_Keystone_5000-5004_Miniature, symbol Connector:TestPoint
- removed TP21: HALL_SWITCH, TestPoint:TestPoint_Keystone_5000-5004_Miniature, symbol Connector:TestPoint
- removed U5: A3214ELHLT-T, Package_TO_SOT_SMD:SOT-23W_Handsoldering, symbol Sensor_Magnetic:A3214ELHLT-T
Connections:
- wire segments 174 -> 156
Other:
- note added: "CONNECTORS\nTEENSY LC: Qty 2, 14 pins each side (does not include end/center pins)\nFEATHER: one row 12 pins, one row 16 pins"
- note removed: "NOTES:\nv0.2 represents improvements learned from producing v0.1, along witih some additional best\npractices (decoupling caps, series LED matrix signal resistor and large power filter cap).\nv0.2 was not produced, but it should work well."
- moved on the sheet: C3, C4, H1

Commit message: Core logic board split to 5 sheets, power/driver sheet draft, pcb draft.
Parts:
- removed C1: 0.1uF, Capacitor_SMD:C_0805_2012Metric, symbol Device:CP1_Small
- removed C2: 10uF, Capacitor_SMD:C_0805_2012Metric, symbol Device:CP1_Small
- removed C6: 1000uF, Capacitor_SMD:CP_Elec_8x10, symbol Device:CP1_Small
- removed Q22, Q23: MMBT4401LT1G, Digikey:SOT-23-3, symbol Digikey-Transistors:MMBT4401LT1G
- removed R29, R32, R35: 1K5, Resistor_SMD:R_0805_2012Metric, symbol Device:R
- removed R30, R33: 1K8, Resistor_SMD:R_0805_2012Metric, symbol Device:R
- removed R31, R34: 11, Resistor_SMD:R_0805_2012Metric, symbol Device:R
- removed R36, R37, R38, R39, R40: 10k, Resistor_SMD:R_0805_2012Metric, symbol Device:R
- removed TP10: SENSE1, TestPoint:TestPoint_Keystone_5000-5004_Miniature, symbol Connector:TestPoint
- removed TP11: SENSE2, TestPoint:TestPoint_Keystone_5000-5004_Miniature, symbol Connector:TestPoint
- removed TP12: SENSE_OUT_A, TestPoint:TestPoint_Keystone_5000-5004_Miniature, symbol Connector:TestPoint
- removed TP13: SENSE_OUT_B, TestPoint:TestPoint_Keystone_5000-5004_Miniature, symbol Connector:TestPoint
- removed TP14: SENSE_PULSE, TestPoint:TestPoint_Keystone_5000-5004_Miniature, symbol Connector:TestPoint
- removed TP9: GNDD, TestPoint:TestPoint_Keystone_5000-5004_Miniature, symbol Connector:TestPoint
- removed U3: LM393, Digikey:SOIC-8_W3.9mm, symbol Comparator:LM393
- renumbered C3 to C1, C4 to C2, R28 to R2, R46 to R3, R41 to R4, R42 to R5, R44 to R6, R45 to R7, TP19 to TP10, TP15 to TP11, TP16 to TP12, TP17 to TP13, TP18 to TP14
Connections:
- net LED_MATRIX: now also R3.2; no longer R3.1, TP10.1, U2.15 (17_Vin)
- net V+USB renamed TEENSY_VUSB
- new net: R3.1, TP10.1, U2.15 (17_Vin)
Other:
- note removed: "DNI"
- note removed: "SENSE SIGNAL PROCESSING"
- moved on the sheet: C1, C2, H1, R3, TP10

Commit message: Add I2C bus, clean-up power symbols, update MCU sheet.
Parts:
- removed TP11: +3V3, TestPoint:TestPoint_Keystone_5000-5004_Miniature, symbol Connector:TestPoint
Connections:
- net +3V3: no longer R2.1, U2.31 (3.3V_max100mA), U2.35 (AREF)
- net +VSW: no longer R4.1, U2.33 (Vin)
- net -BATT: no longer R5.2, U2.32 (GND)
- net GNDD: now also R5.2, U2.32 (GND)
- new net TEENSY_3V3: R2.1, U2.31 (3.3V_max100mA), U2.35 (AREF)
- new net TEENSY_VIN: R4.1, U2.33 (Vin)
Other:
- note added: "TO DO: Add Feather module."
- note added: "TO DO: Update this to be SAO, and some easy to add I2C OLED 4-pin header."
- note added: "Teensy LC has incoming USB power/programming on board.\n\n*** CUT THE USB-VIN bridge. ***"
- note added: "Use +3V3 for low power accessories:\nHall sensors, sense circuit, MCU"
- note removed: "Teensy LC has incoming USB\npower/programming on board.\n\nUSB V+ bridge cut and routes ONLY\nto the LiPo charger module.\n\nLiPo must be connected for whole\nsystem to work."
- note removed: "Use +3V3 for low power accessories:\nReed switch, hall sensors, sense circuit, expansion bus, …"
Changed lines of the file:
@@
 	1650 2250 1800 2250
 Wire Wire Line
-	5300 1300 5300 2650
+	5300 1650 5300 2650
 Wire Wire Line
 	5300 2650 3950 2650
-Text GLabel 5000 1250 1    50   Output ~ 0
+Text GLabel 5000 1700 1    50   Output ~ 0
 TEENSY_VUSB
 NoConn ~ 3950 2050
 NoConn ~ 3950 2150
-$Comp
-L power:+VSW #PWR0119
-U 1 1 5D31CDEF
-P 5300 1300
-AR Path="/5E755787/5D31CDEF" Ref="#PWR0119"  Part="1"
-AR Path="/5E755AC8/5D2551FF/5D31CDEF" Ref="#PWR?"  Part="1"
-F 0 "#PWR0119" H 5300 1150 50  0001 C CNN
-F 1 "+VSW" H 5315 1473 50  0000 C CNN
-F 2 "" H 5300 1300 50  0001 C CNN
-F 3 "" H 5300 1300 50  0001 C CNN
-	1    5300 1300
-	1    0    0    -1
-$EndComp
 Wire Wire Line
 	5000 4200 5000 2750
 Wire Wire Line
-	5000 1250 5000 2550
+	5000 1700 5000 2550
 Wire Wire Line
 	5000 2550 3950 2550
 Wire Wire Line
 	5000 2750 3950 2750
-$Comp
-L power:+3V3 #PWR0120
-U 1 1 5D32AA99
-P 6000 1300
-AR Path="/5E755787/5D32AA99" Ref="#PWR0120"  Part="1"
-AR Path="/5E755AC8/5D2551FF/5D32AA99" Ref="#PWR?"  Part="1"
-F 0 "#PWR0120" H 6000 1150 50  0001 C CNN
-F 1 "+3V3" H 6015 1473 50  0000 C CNN
-F 2 "" H 6000 1300 50  0001 C CNN
-F 3 "" H 6000 1300 50  0001 C CNN
-	1    6000 1300
-	1    0    0    -1
-$EndComp
-Wire Wire Line
-	6000 2850 3950 2850
-Wire Wire Line
-	6000 1300 6000 1500
-Wire Wire Line
-	3950 2450 6000 2450
-Connection ~ 6000 2450
-Wire Wire Line
-	6000 2450 6000 2850
+Wire Wire Line
+	5650 2850 3950 2850
+Wire Wire Line
+	3950 2450 5650 2450
+Wire Wire Line
+	5650 2450 5650 2850
 $Comp
 L Device:R R4
@@
 	5300 2650 5300 3250
 Connection ~ 5300 2650
-Text Notes 5250 850  0    50   ~ 0
+Text Notes 4750 1000 0    50   ~ 0
 Battery Voltage Monitor for +VSW\nAnalog reads 1/2 battery voltage
-Text Notes 850  1350 0    50   ~ 0
-Teensy LC has incoming USB\npower/programming on board.\n\nUSB V+ bridge cut and routes ONLY\nto the LiPo charger module.\n\nLiPo must be connected for whole\nsystem to work.
-$Comp
-L power:-BATT #PWR0121
-U 1 1 5D337E9E
-P 5000 4200
-AR Path="/5E755787/5D337E9E" Ref="#PWR0121"  Part="1"
-AR Path="/5E755AC8/5D2551FF/5D337E9E" Ref="#PWR?"  Part="1"
-F 0 "#PWR0121" H 5000 4050 50  0001 C CNN
-F 1 "-BATT" H 5015 4373 50  0000 C CNN
-F 2 "" H 5000 4200 50  0001 C CNN
-F 3 "" H 5000 4200 50  0001 C CNN
-	1    5000 4200
-	-1   0    0    1
-$EndComp
-$Comp
-L power:-BATT #PWR0122
-U 1 1 5D338C7F
-P 5300 4200
-AR Path="/5E755787/5D338C7F" Ref="#PWR0122"  Part="1"
-AR Path="/5E755AC8/5D2551FF/5D338C7F" Ref="#PWR?"  Part="1"
-F 0 "#PWR0122" H 5300 4050 50  0001 C CNN
-F 1 "-BATT" H 5315 4373 50  0000 C CNN
-F 2 "" H 5300 4200 50  0001 C CNN
-F 3 "" H 5300 4200 50  0001 C CNN
-	1    5300 4200
-	-1   0    0    1
-$EndComp
-Text Notes 6250 1150 0    50   ~ 0
-Use +3V3 for low power accessories:\nReed switch, hall sensors, sense circuit, expansion bus, …
+Text Notes 900  900  0    50   ~ 0
+Teensy LC has incoming USB power/programming on board.\n\n*** CUT THE USB-VIN bridge. ***
+Text Notes 5750 1300 0    50   ~ 0
+Use +3V3 for low power accessories:\nHall sensors, sense circuit, MCU
 Text GLabel 7000 3900 2    50   BiDi ~ 0
 I2C_CLOCK
@@
 $EndComp
 $Comp
-L Connector:TestPoint TP11
-U 1 1 5D4D6E00
-P 6300 1500
-AR Path="/5E755787/5D4D6E00" Ref="TP11"  Part="1"
-AR Path="/5E755AC8/5D2551FF/5D4D6E00" Ref="TP?"  Part="1"
-F 0 "TP11" H 6358 1618 50  0000 L CNN
-F 1 "+3V3" H 6358 1527 50  0000 L CNN
-F 2 "TestPoint:TestPoint_Keystone_5000-5004_Miniature" H 6500 1500 50  0001 C CNN
-F 3 "~" H 6500 1500 50  0001 C CNN
-	1    6300 1500
-	1    0    0    -1
-$EndComp
-Wire Wire Line
-	6300 1500 6000 1500
-Connection ~ 6000 1500
-Wire Wire Line
-	6000 1500 6000 2450
-$Comp
 L Connector:TestPoint TP12
 U 1 1 5D4DAE01
@@
 F 3 "~" H 700 2000 50  0001 C CNN
 	1    700  2000
-	1    0    0    -1
-$EndComp
-$Comp
-L power:+3V3 #PWR0130
-U 1 1 5D4CC3D1
-P 700 1850
-AR Path="/5E755787/5D4CC3D1" Ref="#PWR0130"  Part="1"
-AR Path="/5E755AC8/5D2551FF/5D4CC3D1" Ref="#PWR?"  Part="1"
-F 0 "#PWR0130" H 700 1700 50  0001 C CNN
-F 1 "+3V3" H 715 2023 50  0000 C CNN
-F 2 "" H 700 1850 50  0001 C CNN
-F 3 "" H 700 1850 50  0001 C CNN
-	1    700  1850
 	1    0    0    -1
 $EndComp
@@
 Wire Wire Line
 	6050 3500 6050 3950
-Text Notes 1950 1550 0    50   ~ 0
+Text Notes 1650 1550 0    50   ~ 0
 CONNECTORS\nTEENSY LC: Qty 2, 14 pins each side (does not include end/center pins)\nFEATHER: one row 12 pins, one row 16 pins
 Wire Wire Line
@@
 Wire Wire Line
 	1000 3550 1000 4250
+$Comp
+L power:GNDD #PWR?
+U 1 1 5E79D787
+P 5000 4200
+AR Path="/5E755787/5E79D787" Ref="#PWR?"  Part="1"
+AR Path="/5E755AC8/5D2551FF/5E79D787" Ref="#PWR?"  Part="1"
+F 0 "#PWR?" H 5000 3950 50  0001 C CNN
+F 1 "GNDD" H 5004 4045 50  0000 C CNN
+F 2 "" H 5000 4200 50  0001 C CNN
+F 3 "" H 5000 4200 50  0001 C CNN
+	1    5000 4200
+	1    0    0    -1
+$EndComp
+$Comp
+L power:GNDD #PWR?
+U 1 1 5E7A2329
+P 5300 4200
+AR Path="/5E755787/5E7A2329" Ref="#PWR?"  Part="1"
+AR Path="/5E755AC8/5D2551FF/5E7A2329" Ref="#PWR?"  Part="1"
+F 0 "#PWR?" H 5300 3950 50  0001 C CNN
+F 1 "GNDD" H 5304 4045 50  0000 C CNN
+F 2 "" H 5300 4200 50  0001 C CNN
+F 3 "" H 5300 4200 50  0001 C CNN
+	1    5300 4200
+	1    0    0    -1
+$EndComp
+Connection ~ 5650 2450
+Text GLabel 5650 1650 1    50   Input ~ 0
+TEENSY_3V3
+Wire Wire Line
+	5650 1650 5650 2450
+Text GLabel 700  1650 1    50   Input ~ 0
+TEENSY_3V3
+Wire Wire Line
+	700  1850 700  1650
+Text Notes 700  6150 0    50   ~ 10
+TO DO: Update this to be SAO, and some easy to add I2C OLED 4-pin header.
+Text Notes 8050 1350 0    50   ~ 10
+TO DO: Add Feather module.
+Text GLabel 5300 1650 1    50   Input ~ 0
+TEENSY_VIN
 $EndSCHEMATC
