File: Electronic Design/Interactive Core Memory Badge (Logic) v0.3/Interactive Core Memory Badge (Logic) Driver v0.3.sch (KiCad schematic (older format))
At the start: 63 parts, among them J10 SSW-116-22-F-S-VS‎, J9 SSW-116-22-F-S-VS‎, Q10 MMBT4401LT1G, Q11 MMBT4403LT1G, Q12 MMBT4401LT1G, Q13 MMBT4403LT1G, Q14 MMBT4401LT1G, Q15 MMBT4403LT1G, Q16 MMBT4401LT1G, Q17 MMBT4403LT1G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

Commit message: Final push of core board layout v0.3
Connections:
- net at Q2.3 (C): now also D2.3, D4.3
- net at D6.3, D8.3: now also Q7.3 (C)
Other:
- moved on the sheet: Q2, Q7, R14, R8
Changed lines of the file:
@@
 Connection ~ 2100 4950
 Connection ~ 1500 4900
-Text GLabel 900  4250 0    50   Input ~ 0
+Text GLabel 900  4200 0    50   Input ~ 0
 Q1P
 Text GLabel 900  5700 0    50   Input ~ 0
@@
 	900  5700 950  5700
 Wire Wire Line
-	900  4250 950  4250
-Wire Wire Line
-	1250 4250 1400 4250
+	900  4200 950  4200
+Wire Wire Line
+	1250 4200 1400 4200
 Wire Wire Line
 	1250 5700 1400 5700
@@
 L power:VMEM #PWR0132
 U 1 1 5D3B6BE3
-P 1700 4050
-F 0 "#PWR0132" H 1700 3900 50  0001 C CNN
-F 1 "VMEM" H 1715 4223 50  0000 C CNN
-F 2 "" H 1700 4050 50  0001 C CNN
-F 3 "" H 1700 4050 50  0001 C CNN
-	1    1700 4050
+P 1700 4000
+F 0 "#PWR0132" H 1700 3850 50  0001 C CNN
+F 1 "VMEM" H 1715 4173 50  0000 C CNN
+F 2 "" H 1700 4000 50  0001 C CNN
+F 3 "" H 1700 4000 50  0001 C CNN
+	1    1700 4000
 	1    0    0    -1
 $EndComp
@@
 L Digikey-Transistors:MMBT4403LT1G Q7
 U 1 1 5D5BD2C4
-P 4200 4250
-F 0 "Q7" H 4388 4303 60  0000 L CNN
-F 1 "MMBT4403LT1G" H 4388 4197 60  0000 L CNN
-F 2 "Digikey:SOT-23-3" H 4400 4450 60  0001 L CNN
-F 3 "http://www.onsemi.com/pub/Collateral/MMBT4403LT1-D.PDF" H 4400 4550 60  0001 L CNN
-F 4 "MMBT4403LT1GOSCT-ND" H 4400 4650 60  0001 L CNN "Digi-Key_PN"
-F 5 "MMBT4403LT1G" H 4400 4750 60  0001 L CNN "MPN"
-F 6 "Discrete Semiconductor Products" H 4400 4850 60  0001 L CNN "Category"
-F 7 "Transistors - Bipolar (BJT) - Single" H 4400 4950 60  0001 L CNN "Family"
-F 8 "http://www.onsemi.com/pub/Collateral/MMBT4403LT1-D.PDF" H 4400 5050 60  0001 L CNN "DK_Datasheet_Link"
-F 9 "/product-detail/en/on-semiconductor/MMBT4403LT1G/MMBT4403LT1GOSCT-ND/1139820" H 4400 5150 60  0001 L CNN "DK_Detail_Page"
-F 10 "TRANS PNP 40V 0.6A SOT23" H 4400 5250 60  0001 L CNN "Description"
-F 11 "ON Semiconductor" H 4400 5350 60  0001 L CNN "Manufacturer"
-F 12 "Active" H 4400 5450 60  0001 L CNN "Status"
-	1    4200 4250
+P 4200 4200
+F 0 "Q7" H 4388 4253 60  0000 L CNN
+F 1 "MMBT4403LT1G" H 4388 4147 60  0000 L CNN
+F 2 "Digikey:SOT-23-3" H 4400 4400 60  0001 L CNN
+F 3 "http://www.onsemi.com/pub/Collateral/MMBT4403LT1-D.PDF" H 4400 4500 60  0001 L CNN
+F 4 "MMBT4403LT1GOSCT-ND" H 4400 4600 60  0001 L CNN "Digi-Key_PN"
+F 5 "MMBT4403LT1G" H 4400 4700 60  0001 L CNN "MPN"
+F 6 "Discrete Semiconductor Products" H 4400 4800 60  0001 L CNN "Category"
+F 7 "Transistors - Bipolar (BJT) - Single" H 4400 4900 60  0001 L CNN "Family"
+F 8 "http://www.onsemi.com/pub/Collateral/MMBT4403LT1-D.PDF" H 4400 5000 60  0001 L CNN "DK_Datasheet_Link"
+F 9 "/product-detail/en/on-semiconductor/MMBT4403LT1G/MMBT4403LT1GOSCT-ND/1139820" H 4400 5100 60  0001 L CNN "DK_Detail_Page"
+F 10 "TRANS PNP 40V 0.6A SOT23" H 4400 5200 60  0001 L CNN "Description"
+F 11 "ON Semiconductor" H 4400 5300 60  0001 L CNN "Manufacturer"
+F 12 "Active" H 4400 5400 60  0001 L CNN "Status"
+	1    4200 4200
 	1    0    0    -1
 $EndComp
@@
 Wire Wire Line
 	3500 4850 5350 4850
-Text GLabel 3500 4250 0    50   Input ~ 0
+Text GLabel 3500 4200 0    50   Input ~ 0
 Q2P
 Text GLabel 3500 5700 0    50   Input ~ 0
@@
 	3500 5700 3550 5700
 Wire Wire Line
-	3500 4250 3550 4250
+	3500 4200 3550 4200
 $Comp
 L Device:R R14
 U 1 1 5D5BD310
-P 3700 4250
-F 0 "R14" V 3493 4250 50  0000 C CNN
-F 1 "470" V 3584 4250 50  0000 C CNN
-F 2 "Resistor_SMD:R_0805_2012Metric" V 3630 4250 50  0001 C CNN
-F 3 "~" H 3700 4250 50  0001 C CNN
-	1    3700 4250
+P 3700 4200
+F 0 "R14" V 3493 4200 50  0000 C CNN
+F 1 "470" V 3584 4200 50  0000 C CNN
+F 2 "Resistor_SMD:R_0805_2012Metric" V 3630 4200 50  0001 C CNN
+F 3 "~" H 3700 4200 50  0001 C CNN
+	1    3700 4200
 	0    1    1    0
 $EndComp
 Wire Wire Line
-	3850 4250 4000 4250
+	3850 4200 4000 4200
 $Comp
 L Device:R R15
@@
 L power:VMEM #PWR0136
 U 1 1 5D5BD324
-P 4300 4050
-F 0 "#PWR0136" H 4300 3900 50  0001 C CNN
-F 1 "VMEM" H 4315 4223 50  0000 C CNN
-F 2 "" H 4300 4050 50  0001 C CNN
-F 3 "" H 4300 4050 50  0001 C CNN
-	1    4300 4050
+P 4300 4000
+F 0 "#PWR0136" H 4300 3850 50  0001 C CNN
+F 1 "VMEM" H 4315 4173 50  0000 C CNN
+F 2 "" H 4300 4000 50  0001 C CNN
+F 3 "" H 4300 4000 50  0001 C CNN
+	1    4300 4000
 	1    0    0    -1
 $EndComp
@@
 L Device:R R8
 U 1 1 5D48D653
-P 1100 4250
-F 0 "R8" V 893 4250 50  0000 C CNN
-F 1 "470" V 984 4250 50  0000 C CNN
-F 2 "Resistor_SMD:R_0805_2012Metric" V 1030 4250 50  0001 C CNN
-F 3 "~" H 1100 4250 50  0001 C CNN
-	1    1100 4250
+P 1100 4200
+F 0 "R8" V 893 4200 50  0000 C CNN
+F 1 "470" V 984 4200 50  0000 C CNN
+F 2 "Resistor_SMD:R_0805_2012Metric" V 1030 4200 50  0001 C CNN
+F 3 "~" H 1100 4200 50  0001 C CNN
+	1    1100 4200
 	0    1    1    0
 $EndComp
@@
 L Digikey-Transistors:MMBT4403LT1G Q2
 U 1 1 5D49119D
-P 1600 4250
-F 0 "Q2" H 1788 4303 60  0000 L CNN
-F 1 "MMBT4403LT1G" H 1788 4197 60  0000 L CNN
-F 2 "Digikey:SOT-23-3" H 1800 4450 60  0001 L CNN
-F 3 "http://www.onsemi.com/pub/Collateral/MMBT4403LT1-D.PDF" H 1800 4550 60  0001 L CNN
-F 4 "MMBT4403LT1GOSCT-ND" H 1800 4650 60  0001 L CNN "Digi-Key_PN"
-F 5 "MMBT4403LT1G" H 1800 4750 60  0001 L CNN "MPN"
-F 6 "Discrete Semiconductor Products" H 1800 4850 60  0001 L CNN "Category"
-F 7 "Transistors - Bipolar (BJT) - Single" H 1800 4950 60  0001 L CNN "Family"
-F 8 "http://www.onsemi.com/pub/Collateral/MMBT4403LT1-D.PDF" H 1800 5050 60  0001 L CNN "DK_Datasheet_Link"
-F 9 "/product-detail/en/on-semiconductor/MMBT4403LT1G/MMBT4403LT1GOSCT-ND/1139820" H 1800 5150 60  0001 L CNN "DK_Detail_Page"
-F 10 "TRANS PNP 40V 0.6A SOT23" H 1800 5250 60  0001 L CNN "Description"
-F 11 "ON Semiconductor" H 1800 5350 60  0001 L CNN "Manufacturer"
-F 12 "Active" H 1800 5450 60  0001 L CNN "Status"
-	1    1600 4250
+P 1600 4200
+F 0 "Q2" H 1788 4253 60  0000 L CNN
+F 1 "MMBT4403LT1G" H 1788 4147 60  0000 L CNN
+F 2 "Digikey:SOT-23-3" H 1800 4400 60  0001 L CNN
+F 3 "http://www.onsemi.com/pub/Collateral/MMBT4403LT1-D.PDF" H 1800 4500 60  0001 L CNN
+F 4 "MMBT4403LT1GOSCT-ND" H 1800 4600 60  0001 L CNN "Digi-Key_PN"
+F 5 "MMBT4403LT1G" H 1800 4700 60  0001 L CNN "MPN"
+F 6 "Discrete Semiconductor Products" H 1800 4800 60  0001 L CNN "Category"
+F 7 "Transistors - Bipolar (BJT) - Single" H 1800 4900 60  0001 L CNN "Family"
+F 8 "http://www.onsemi.com/pub/Collateral/MMBT4403LT1-D.PDF" H 1800 5000 60  0001 L CNN "DK_Datasheet_Link"
+F 9 "/product-detail/en/on-semiconductor/MMBT4403LT1G/MMBT4403LT1GOSCT-ND/1139820" H 1800 5100 60  0001 L CNN "DK_Detail_Page"
+F 10 "TRANS PNP 40V 0.6A SOT23" H 1800 5200 60  0001 L CNN "Description"
+F 11 "ON Semiconductor" H 1800 5300 60  0001 L CNN "Manufacturer"
+F 12 "Active" H 1800 5400 60  0001 L CNN "Status"
+	1    1600 4200
 	1    0    0    -1
 $EndComp
@@
 CORE ARRAY ENABLE
 Wire Wire Line
-	3800 4450 5000 4450
-Wire Wire Line
-	1200 4450 2400 4450
+	3800 4450 4300 4450
+Wire Wire Line
+	1200 4450 1700 4450
 Text GLabel 2450 2300 0    50   Output ~ 0
 XB3
@@
 Wire Wire Line
 	1250 7100 1900 7100
+Wire Wire Line
+	1700 4400 1700 4450
+Connection ~ 1700 4450
+Wire Wire Line
+	1700 4450 2400 4450
+Wire Wire Line
+	4300 4400 4300 4450
+Connection ~ 4300 4450
+Wire Wire Line
+	4300 4450 5000 4450
 $EndSCHEMATC

Commit message: V0.3 Logic Board released for prototype!
Parts:
- renumbered C12 to C8, J9 to J6, J10 to J7
Changed lines of the file:
@@
 Sheet 2 5
 Title "Core 64 - Core Array Driver"
-Date "2020-04-24"
+Date "2020-05-18"
 Rev "0.3"
 Comp "Andy Geppert - Machine Ideas, LLC"
@@
 L power:GNDPWR #PWR0134
 U 1 1 5D3EAB15
-P 3950 2250
-F 0 "#PWR0134" H 3950 2050 50  0001 C CNN
-F 1 "GNDPWR" H 3954 2096 50  0000 C CNN
-F 2 "" H 3950 2200 50  0001 C CNN
-F 3 "" H 3950 2200 50  0001 C CNN
-	1    3950 2250
+P 3950 2300
+F 0 "#PWR0134" H 3950 2100 50  0001 C CNN
+F 1 "GNDPWR" H 3954 2146 50  0000 C CNN
+F 2 "" H 3950 2250 50  0001 C CNN
+F 3 "" H 3950 2250 50  0001 C CNN
+	1    3950 2300
 	1    0    0    -1
 $EndComp
@@
 	2450 2600 2550 2600
 $Comp
-L Connector:Conn_01x16_Female J10
+L Connector:Conn_01x16_Female J7
 U 1 1 5E78B5ED
 P 2750 2300
-F 0 "J10" H 1950 3250 50  0000 C CNN
+F 0 "J7" H 1950 3250 50  0000 C CNN
 F 1 "SSW-116-22-F-S-VS‎" H 2350 3150 50  0000 C CNN
 F 2 "Connector_PinHeader_2.54mm:PinHeader_1x16_P2.54mm_Vertical_SMD_and_TH_Pin1Left" H 2750 2300 50  0001 C CNN
@@
 $EndComp
 $Comp
-L Connector:Conn_01x16_Female J9
+L Connector:Conn_01x16_Female J6
 U 1 1 5E78B5F3
 P 550 2300
-F 0 "J9" H 500 3250 50  0000 C CNN
+F 0 "J6" H 500 3250 50  0000 C CNN
 F 1 "SSW-116-22-F-S-VS‎" H 100 3150 50  0000 C CNN
 F 2 "Connector_PinHeader_2.54mm:PinHeader_1x16_P2.54mm_Vertical_SMD_and_TH_Pin1Left" H 550 2300 50  0001 C CNN
@@
 AR Path="/5E755787/5E91F406" Ref="C?"  Part="1"
 AR Path="/5E755AC8/5D2551FF/5E91F406" Ref="C?"  Part="1"
-AR Path="/5E755AC8/5E91F406" Ref="C12"  Part="1"
-F 0 "C12" H 1350 7400 50  0000 L CNN
+AR Path="/5E755AC8/5E91F406" Ref="C8"  Part="1"
+F 0 "C8" H 1350 7400 50  0000 L CNN
 F 1 "1000uF" H 1350 7300 50  0000 L CNN
 F 2 "Capacitor_SMD:CP_Elec_10x10" H 1250 7300 50  0001 C CNN
@@
 Wire Wire Line
 	4300 4450 5000 4450
+Wire Wire Line
+	3950 2250 3950 2300
 $EndSCHEMATC
