File: Electronic Design/Core64 LB v0.4/Core64 LB v0.4 Power.sch (KiCad schematic (older format))
At the start: 16 parts, among them J2 Conn_01x02_Male, J3 Conn_01x08_Female, SW1 JS102011SAQN, U1 LD1117S33TR_SOT223

Commit message: Correct Logic Board filenames to LB from CB
Parts:
- gave numbers to parts that had none: 5
Changed lines of the file:
@@
 EESchema Schematic File Version 4
-LIBS:Core64 CB v0.4-cache
+LIBS:Core64 LB v0.4-cache
 EELAYER 29 0
 EELAYER END
@@
 VSW_HALF_VOL_MONITOR
 $Comp
-L Transistor_FET:IRLML2060 Q?
+L Transistor_FET:IRLML2060 Q22
 U 1 1 5E770BB5
 P 1850 6650
-F 0 "Q?" V 2101 6650 50  0000 C CNN
+F 0 "Q22" V 2101 6650 50  0000 C CNN
 F 1 "IRLML6344TRPBF" V 2194 6650 50  0000 C CNN
 F 2 "Digikey:SOT-23-3" H 2050 6575 50  0001 L CIN
@@
 ALTERNATE CONNECTOR - Generic SMT 2-pin .1” \nheader option for everything else.
 $Comp
-L BM03B-PASS-1-TFT__LF__SN_:BM03B-PASS-1-TFT__LF__SN_ J?
+L BM03B-PASS-1-TFT__LF__SN_:BM03B-PASS-1-TFT__LF__SN_ J8
 U 1 1 5E870E95
 P 1800 2550
-F 0 "J?" H 2250 2800 50  0000 C CNN
+F 0 "J8" H 2250 2800 50  0000 C CNN
 F 1 "BM03B-PASS-1-TFT__LF__SN_" H 2200 2700 50  0000 C CNN
 F 2 "JST_BM03B-PASS-1-TFT:BM03BPASS1TFTLFSN" H 2550 2650 50  0001 L CNN
@@
 	1800 2550 2400 2550
 $Comp
-L Diode:MBR0520 D?
+L Diode:MBR0520 D13
 U 1 1 5E87F7F2
 P 3400 4800
-F 0 "D?" H 3400 4581 50  0000 C CNN
+F 0 "D13" H 3400 4581 50  0000 C CNN
 F 1 "MBR120" H 3400 4674 50  0000 C CNN
 F 2 "Diode_SMD:D_SOD-123F" H 3400 4625 50  0001 C CNN
@@
 	1000 4900 2350 4900
 $Comp
-L Mechanical:MountingHole_Pad H?
+L Mechanical:MountingHole_Pad H2
 U 1 1 5E8DC4AA
 P 3350 6450
-F 0 "H?" H 3450 6500 50  0000 L CNN
+F 0 "H2" H 3450 6500 50  0000 L CNN
 F 1 "GND PAD" H 3450 6407 50  0000 L CNN
 F 2 "MountingHole:MountingHole_2.2mm_M2_Pad_Via" H 3350 6450 50  0001 C CNN
@@
 	3350 6550 3350 6750
 $Comp
-L Mechanical:MountingHole_Pad H?
+L Mechanical:MountingHole_Pad H1
 U 1 1 5E8DD364
 P 700 6450
-F 0 "H?" H 800 6500 50  0000 L CNN
+F 0 "H1" H 800 6500 50  0000 L CNN
 F 1 "-BATT PAD" H 800 6407 50  0000 L CNN
 F 2 "MountingHole:MountingHole_2.2mm_M2_Pad_Via" H 700 6450 50  0001 C CNN

Commit message: Swap in Teensy 3.2 from LC, set schematic sheet sizes to A, update power schematic
Parts:
- removed D13: MBR120, Diode_SMD:D_SOD-123F, symbol Diode:MBR0520
- removed F1: Polyfuse, Fuse:Fuse_0805_2012Metric, symbol Device:Polyfuse
- removed Q22: IRLML6344TRPBF, Digikey:SOT-23-3, symbol Transistor_FET:IRLML2060
- added C6: 0.1uF, symbol Device:C
- added D13: D_Zener, symbol Device:D_Zener
- added JP1: SolderJumper_2_Bridged, symbol Jumper:SolderJumper_2_Bridged
- added JP?: Current Mon., symbol Jumper:SolderJumper_2_Bridged
- added Q22: BSS315PH6327XTSA1, Digikey:SOT-23-3, symbol Device:Q_PMOS_DGS
- H1: value -BATT PAD -> GND PAD
- R43: value 0.001 -> 100k
- R51: value 10k -> 11k
- R52: value 10k -> 33k
Connections:
- net labels added: 5V0, RPP, V_MON
- net labels removed: 5V_USB, CUR_HI, TEENSY_GND, TEENSY_VIN, VSW_HALF_VOL_MONITOR
- wire segments 71 -> 75
Other:
- note added: "1%"
- note added: "5V POWER SUPPLY"
- note added: "7V MAX !!!"
- note added: "ALL SYSTEM STAR GROUNDING"
- note added: "Cut SJ if you want the \nOFF position to not\nbe powered from\nTeensy USB connector."
- note added: "D"
- note added: "G"
- note added: "OPTIONAL:\n1) Open SJ\n2) Insert 0.01 Ohm\n -or-\n2) Measure current\nbetween RPP & +VSW"
- note added: "POWER SWITCH, RPP, VOLTAGE & CURRENT MONITOR"
- note added: "REVERSE POLARITY PROTECTION\nHIGH SIDE\nhttps://hackaday.com/2011/12/06/reverse-voltage-protection-with-a-p-fet/\nLOW SIDE\nhttps://www.instructables.com/id/Reverse-polarity-protection-for-your-circuit-with/\nIRLML6344TRPBF https://www.digikey.com/product-detail/en/infineon-technologies/IRLML6344TRPBF/IRLML6344TRPBFCT-ND/2538168"
- note added: "S"
- note added: "SILKSCREEN:"
- note added: "SILKSCREEN: ON (BAT) / OFF (USB)"
- note added: "TEENSY 3.2 WITH ALKALINE/NIMH BATTERY PACK\n*** MUST CUT VIN-VUSB TRACE ON TEENSY ***\nTHIS IS THE STANDARD MANUFACTURED KIT CONFIGURATION"
- note removed: "ALL SYSTEM\nSTAR GROUNDING"
- note removed: "BOTH MODES REQUIRE:\nVIN must be supplied TO the Teensy\n(because VIN-VUSB is cut) and the \nCore 64 Logic Board provides it here."
- note removed: "POWER SWITCH, POWER PROTECTION, VOLTAGE & CURRENT MONITOR"
- note removed: "REVERSE POLARITY DETECTION AND SYSTEM\nCURRENT MEASUREMENT CLOSE TO BATTERY.\n\nREF: https://www.instructables.com/id/Reverse-polarity-protection-for-your-circuit-with/\nIRLML6344TRPBF https://www.digikey.com/product-detail/en/infineon-technologies/IRLML6344TRPBF/IRLML6344TRPBFCT-ND/2538168"
- note removed: "REVERSE POLARITY\nPROTECTION"
- note removed: "Reverse polarity protection"
- note removed: "TEENSY LC OR 3.2 AND ALKALINE/NIMH BATTERY PACK\n*** MUST CUT VIN-VUSB TRACE ON TEENSY ***\nTHIS IS THE STANDARD MANUFACTURED KIT CONFIGURATION"
- moved on the sheet: C1, C2, C3, H1, H2, J2, J3, R51, R52, SW1

Commit message: Add regulator and battery connector data sheets, footprints, symbols
Parts:
- removed C1: 1000uF, Capacitor_SMD:CP_Elec_10x10, symbol Device:CP1_Small
- removed C6: 0.1uF, symbol Device:C
- removed D13: D_Zener, symbol Device:D_Zener
- removed J8: BM03B-PASS-1-TFT__LF__SN_, JST_BM03B-PASS-1-TFT:BM03BPASS1TFTLFSN, symbol BM03B-PASS-1-TFT__LF__SN_:BM03B-PASS-1-TFT__LF__SN_
- removed R43: 100k, Resistor_SMD:R_0805_2012Metric, symbol Device:R
- removed U1: LD1117S33TR_SOT223, Package_TO_SOT_SMD:SOT-223-3_TabPin2, symbol Regulator_Linear:LD1117S33TR_SOT223
- added C12, C14: 1uF, Capacitor_SMD:C_0805_2012Metric, symbol Device:C
- added C13, C7: ?uF, Capacitor_SMD:C_0805_2012Metric, symbol Device:C
- added IC1: NCP176AMX330TCG, NCP176AMX330TCG:NCP176AMX330TCG, symbol NCP176AMX330TCG:NCP176AMX330TCG
- added IC2: TPS7A0533PDBVR, TPS7A0533PDBVR:SOT95P280X145-5N, symbol TPS7A0533PDBVR:TPS7A0533PDBVR
- added IC3: LP3961EMP-5.0, LP3961EMP-5.0:SOT150P696X180-5N, symbol LP3961EMP-5.0:LP3961EMP-5.0
- added J8: S03B-PASK-2_LF__SN_, JST_S03B-PASK-2_LF__SN_:S03BPASK2LFSN, symbol S03B-PASK-2_LF__SN_:S03B-PASK-2_LF__SN_
- added J9: JST-PH 2-PIN, Connector_JST:JST_PH_S2B-PH-SM4-TB_1x02-1MP_P2.00mm_Horizontal, symbol Connector:Conn_01x02_Male
- added JP5: Opt. Zen., Jumper:SolderJumper-2_P1.3mm_Open_Pad1.0x1.5mm, symbol Jumper:SolderJumper_2_Open
- added JP6: Opt. Cap., Jumper:SolderJumper-2_P1.3mm_Open_Pad1.0x1.5mm, symbol Jumper:SolderJumper_2_Open
- added JP7: Opt. Res., Jumper:SolderJumper-2_P1.3mm_Bridged_Pad1.0x1.5mm, symbol Jumper:SolderJumper_2_Bridged
- added JP8: Teensy_Charge_Enable, Jumper:SolderJumper-2_P1.3mm_Bridged_Pad1.0x1.5mm, symbol Jumper:SolderJumper_2_Bridged
- added JP9: 3V3_Select, Jumper:SolderJumper-3_P1.3mm_Open_Pad1.0x1.5mm, symbol Jumper:SolderJumper_3_Open
- added R?: 10k, Resistor_SMD:R_0805_2012Metric, symbol Device:R
- added U6: Micro_LiPo_Charger, Core_Memory_8x8_Array:Micro_LiPo_Charger, symbol CORE_64_LIBRARY:Micro_LiPo_Charger
- C2: value 0.1uF -> 1uF; symbol Device:CP1_Small -> Device:C
- C3: value 10uF -> 1uF; symbol Device:CP1_Small -> Device:C
- J2: value Conn_01x02_Male -> 0.1\" 2-PIN
- JP1: value SolderJumper_2_Bridged -> USB_Power_Enable; footprint (none) -> Jumper:SolderJumper-2_P1.3mm_Bridged_Pad1.0x1.5mm
- JP2: renamed from JP?; value Current Mon. -> Opt. Cur. Mon.; footprint (none) -> Jumper:SolderJumper-2_P1.3mm_Bridged_Pad1.0x1.5mm
- R51: value 11k -> 33k
- R52: value 33k -> 11k
Connections:
- net labels added: 3V3
- net labels removed: 3V3_800mA
- wire segments 75 -> 110
- no-connect marks 3 -> 0
Other:
- note added: "*** ALL CONFIGURATIONS REQUIRED CUTTING VIN-VUSB TRACE ON TEENSY ***"
- note added: "1S ONLY !!!"
- note added: "7.5V MAX !!!"
- note added: "ALTERNATE 1S LIPO BATTERY - USER SUPPLIED"
- note added: "ALTERNATE CONNECTOR - JST-PH 2-PIN SMT\nAdafruit 1769 Right Angle Battery Cable Socket\nJST S2B-PH-SM4-TB(LF)(SN), Digi-Key 455-1749-1-ND"
- note added: "ALTERNATE CONNECTOR\nGeneric 2-pin header 0.1”"
- note added: "All non-polarized capacitors are ceramic unless otherwise noted."
- note added: "Alternate, larger"
- note added: "Must\nSelect\nOne"
- note added: "OPT: Open SJ to\ndisable charging\nfrom Teensy USB."
- note added: "OPTIONAL CUR. MON.:\n1) Open Cur. Mon. SJ\n2) Insert 0.01 Ohm\n -or-\n2) Ammeter current\nbetween RPP & +VSW"
- note added: "OPTIONAL FET PROTECT:\n1) .1uF Cap. on left\n2) 100k Res. on bottom\n3) 10V Zener on right"
- note added: "OPTIONAL USB BYPASS:\nAs shipped, switch in\nOFF position connects\nto USB power through\nthe Teensy.\nOPTIONAL:\nCut SJ if you want the \nOFF position to not\nbe powered from\nTeensy USB connector."
- note added: "P-FET"
- note added: "POWER SWITCH, RPP, V & I MONITOR"
- note added: "Preferred, TINY"
- note added: "SILKSCREEN: +/- pins"
- note added: "SOURCE 1 “ON (BAT)”\n BUILT-IN BATTERY PACK (Keystone 2482CN) WITH 4X “AAA” Primary/Alkaline Cells\n OK to use Energizer Ultimate Lithium (light weight!) with open cell 7.2V, loaded will be <7V.\n Battery Pack includes wires and 3-pin plug.\n \n Socket: TH, Side Entry, JST PA S03B-PASK-2(LF)(SN), Digikey 455-1848-ND ($0.44/ea)\n Socket: SMT, Top Entry, JST PA BM03B-PASS-1-TFT(LF)(SN), Digikey 455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"
- note added: "SOURCE 2 “OFF (USB)”\n USB 5V supplied through Teensy 3.2 \n With the VIN-VUSB trace cut on the back of the Teensy, the TEENSY_5VUSB\n is routed directly from the USB Port, to the VUSB pin on the back \n of the Teensy, over to one side of the SPDT switch. In this position\n the VUSB goes back to the Teensy through the 5V regulator."
- note added: "STANDARD MANUFACTURED KIT CONFIGURATION"
- note added: "TWO OPTIONS\n\n1) 1S LiPo + Charger (most convenient)\n A) Choose a 1S Lipo with built-in cell over/under voltage protection. Recommended \n B) Choose a charger. The logic board is designed to accept this one: https://www.adafruit.com/product/1904\n C) 4-pin header to connector charger to the logic board. Or solder direct to logic board.\n\n2) 1S LiPo only (flexible, choose your own connector)\n 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"
- note added: "TWO POWER INPUT SOURCES SELECTED BY SPDT SWITCH"
- note removed: "7V MAX !!!"
- note removed: "ALTERNATE CONNECTOR - Generic SMT 2-pin .1” \nheader option for everything else."
- note removed: "Cut SJ if you want the \nOFF position to not\nbe powered from\nTeensy USB connector."
- note removed: "HACKER POWER OPTION: ADAFRUIT FEATHER WITH REQUIRED LIPO\n*** MUST REMOVE ALKALINE/NIMH BATTERY PACK ***\nUSER MODIFICATION REQUIRED"
- note removed: "HACKER UPGRADE TO USE FEATHER-TEENSY ADAPTER BOARD REQUIRES:\nA) REPLACE THE ALKALINE/NIMH BATTERY PACK WITH 1S LIPO IN THE SAME POWER PORT, OR THE ALTERNATE PORT.\n -or-\nB) REMOVE THE ALKALINE/NIMH BATTERY PACK AND CONNECT 1S LIPO DIRECTLY TO FEATHER JST-PH BATTERY/CHARGING PORT."
- note removed: "MODE 1\n BUILT-IN BATTERY PACK (Keystone 2482CN) WITH 4X “AAA” ALKALINE OR NIMH CELLS\n …or 3-4 “AA” alkaline/NiMh, or 1S LiPo, but the logic board does not recharge these batteries automatically from USB power.\n CONNECTED TO 3 PIN input for Battery Pack\n On PCB: SMT CONN, 3 TERM, HORZ, 2mm spacing, detent lock\n Such as: Keystone 976, JST PA BM03B-PASS-1-TFT(LF)(SN), Adafruit 4391 (JST PH 3-pi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"
- note removed: "MODE 2\n USB 5V through Teensy LC or 3.2 \n VUSB is 5V from USB cable."
- note removed: "OPTIONAL:\n1) Open SJ\n2) Insert 0.01 Ohm\n -or-\n2) Measure current\nbetween RPP & +VSW"
- note removed: "PLACE\nCAPACITOR\nNEAR\nLED MATRIX"
- note removed: "POWER SWITCH, RPP, VOLTAGE & CURRENT MONITOR"
- note removed: "REVERSE POLARITY PROTECTION\nHIGH SIDE\nhttps://hackaday.com/2011/12/06/reverse-voltage-protection-with-a-p-fet/\nLOW SIDE\nhttps://www.instructables.com/id/Reverse-polarity-protection-for-your-circuit-with/\nIRLML6344TRPBF https://www.digikey.com/product-detail/en/infineon-technologies/IRLML6344TRPBF/IRLML6344TRPBFCT-ND/2538168"
- note removed: "SILKSCREEN:"
- note removed: "TEENSY 3.2 WITH ALKALINE/NIMH BATTERY PACK\n*** MUST CUT VIN-VUSB TRACE ON TEENSY ***\nTHIS IS THE STANDARD MANUFACTURED KIT CONFIGURATION"
- note removed: "TO DO: Choose BIG CAP footprint"
- note removed: "TWO POWER MODES SELECTED BY DOUBLE-THROW SWITCH:"
- moved on the sheet: H1, H2, J2, J3, JP1, JP2, Q22, R51, R52, SW1

Commit message: Complete LB power schematic, add 3-to-8 decoder
Parts:
- added R1: 10k, Resistor_SMD:R_0805_2012Metric, symbol Device:R
- C13: value ?uF -> 68uF; footprint Capacitor_SMD:C_0805_2012Metric -> Capacitor_SMD:C_1206_3216Metric
- C7: value ?uF -> 470uF; footprint Capacitor_SMD:C_0805_2012Metric -> Capacitor_SMD:CP_Elec_10x10; symbol Device:C -> Device:CP1; Digikey (none) -> 565-EMHL100ARA471MHA0GCT-ND
- JP9: footprint Jumper:SolderJumper-3_P1.3mm_Open_Pad1.0x1.5mm -> Jumper:SolderJumper-3_P1.3mm_Open_Pad1.0x1.5mm_NumberLabels
- R43: renamed from R?; value 10k -> 100k
Connections:
- net +VSW: now also C13.1, IC3.2 (VIN), R43.1, R1.1
- net -BATT: now also C13.2, C7.2, IC3.4 (~ERROR), IC3.5 (GND), R43.2
- net 5V0: now also C7.1, IC3.3 (VOUT)
- net at IC3.1 (~SD): now also R1.2
Other:
- note added: "0.2Ω ≤ COUT ESR ≤ 5Ω"
- note added: "All non-polarized capacitors are X7R or X5R ceramic unless otherwise noted."
- note added: "CIN ESR (mΩ) / CIN (μF) ≤ 1.5\nX7R or X5R Ceramic"
- note added: "See data sheet for\ncapacitor requirements"
- note removed: "All non-polarized capacitors are ceramic unless otherwise noted."
- moved on the sheet: C13, IC3, R43
Changed lines of the file:
@@
 Text Notes 9300 6550 2    50   ~ 0
 HIGH POWER SYSTEM GROUND
-Text Notes 5650 4550 0    50   ~ 0
+Text Notes 5800 4550 0    50   ~ 0
 LED ARRAY, TEENSY VIN
 $Comp
@@
 Text GLabel 4100 5250 2    50   Output ~ 0
 +VSW
-Text GLabel 4900 4800 1    50   Input ~ 0
+Text GLabel 5000 4800 0    50   Input ~ 0
 +VSW
 $Comp
 L power:GND #PWR0113
 U 1 1 5F56E724
-P 5500 6400
+P 6050 5850
 AR Path="/5E7548ED/5F56E724" Ref="#PWR0113"  Part="1"
 AR Path="/5E755AC8/5D254AE8/5F56E724" Ref="#PWR?"  Part="1"
-F 0 "#PWR0113" H 5500 6150 50  0001 C CNN
-F 1 "GND" H 5505 6225 50  0000 C CNN
-F 2 "" H 5500 6400 50  0001 C CNN
-F 3 "" H 5500 6400 50  0001 C CNN
-	1    5500 6400
-	1    0    0    -1
-$EndComp
-Text Notes 5850 6550 0    50   ~ 0
+F 0 "#PWR0113" H 6050 5600 50  0001 C CNN
+F 1 "GND" H 6055 5675 50  0000 C CNN
+F 2 "" H 6050 5850 50  0001 C CNN
+F 3 "" H 6050 5850 50  0001 C CNN
+	1    6050 5850
+	1    0    0    -1
+$EndComp
+Text Notes 5550 6150 0    50   ~ 0
 HIGH POWER SYSTEM GROUND
 Connection ~ 3850 5550
@@
 Text Notes 2900 6050 0    50   ~ 0
 OPTIONAL CUR. MON.:\n1) Open Cur. Mon. SJ\n2) Insert 0.01 Ohm\n    -or-\n2) Ammeter current\nbetween RPP & +VSW
-Text Notes 4850 4450 0    118  ~ 0
+Text Notes 5000 4450 0    118  ~ 0
 5V POWER SUPPLY
 Wire Wire Line
 	2900 4950 3000 4950
-Text GLabel 7150 4600 2    50   Output ~ 0
+Text GLabel 7200 4800 2    50   Output ~ 0
 5V0
 Text GLabel 5100 7450 1    50   Input ~ 0
@@
 	6400 3300 6500 3300
 Text Notes 6300 6750 0    50   ~ 0
-All non-polarized capacitors are ceramic unless otherwise noted.
+All non-polarized capacitors are X7R or X5R ceramic unless otherwise noted.
 $Comp
 L NCP176AMX330TCG:NCP176AMX330TCG IC1
@@
 Text Notes 8550 4650 0    50   ~ 0
 Alternate, larger
-Wire Wire Line
-	7900 5850 7900 5950
 $Comp
 L power:GND #PWR0119
@@
 Connection ~ 7900 5950
 Wire Wire Line
-	7900 5950 7900 6100
-Wire Wire Line
 	7750 6300 7750 6350
 Wire Wire Line
@@
 	8300 5200 8350 5200
 Connection ~ 8300 5000
-Wire Wire Line
-	8300 4700 8300 4800
 Connection ~ 8300 4800
 Wire Wire Line
@@
 F 0 "JP9" V 9750 5650 50  0000 L CNN
 F 1 "3V3_Select" V 9600 5100 50  0000 L CNN
-F 2 "Jumper:SolderJumper-3_P1.3mm_Open_Pad1.0x1.5mm" H 9850 5550 50  0001 C CNN
+F 2 "Jumper:SolderJumper-3_P1.3mm_Open_Pad1.0x1.5mm_NumberLabels" H 9850 5550 50  0001 C CNN
 F 3 "~" H 9850 5550 50  0001 C CNN
 	1    9850 5550
@@
 Text Notes 10000 6150 0    50   ~ 0
 Must\nSelect\nOne
-Text GLabel 8300 4700 1    50   Input ~ 0
+Text GLabel 8200 4650 0    50   Input ~ 0
 5V0
-Text GLabel 7900 5850 1    50   Input ~ 0
+Text GLabel 7850 5750 0    50   Input ~ 0
 5V0
 $Comp
-L Device:C C?
+L Device:CP1 C?
 U 1 1 5F69BA6F
-P 7450 4850
+P 7100 5250
 AR Path="/5E755787/5F69BA6F" Ref="C?"  Part="1"
 AR Path="/5E755AC8/5D2551FF/5F69BA6F" Ref="C?"  Part="1"
 AR Path="/5EA63449/5F69BA6F" Ref="C?"  Part="1"
 AR Path="/5E7548ED/5F69BA6F" Ref="C7"  Part="1"
-F 0 "C7" H 7541 4896 50  0000 L CNN
-F 1 "?uF" H 7541 4805 50  0000 L CNN
-F 2 "Capacitor_SMD:C_0805_2012Metric" H 7450 4850 50  0001 C CNN
-F 3 "~" H 7450 4850 50  0001 C CNN
-	1    7450 4850
-	-1   0    0    -1
+F 0 "C7" H 7191 5296 50  0000 L CNN
+F 1 "470uF" H 7191 5205 50  0000 L CNN
+F 2 "Capacitor_SMD:CP_Elec_10x10" H 7100 5250 50  0001 C CNN
+F 3 "" H 7100 5250 50  0001 C CNN
+F 4 "565-EMHL100ARA471MHA0GCT-ND" H 7100 5250 50  0001 C CNN "Digikey"
+	1    7100 5250
+	1    0    0    -1
 $EndComp
 $Comp
 L Device:C C?
 U 1 1 5F69C890
-P 4900 5150
+P 5100 5400
 AR Path="/5E755787/5F69C890" Ref="C?"  Part="1"
 AR Path="/5E755AC8/5D2551FF/5F69C890" Ref="C?"  Part="1"
 AR Path="/5EA63449/5F69C890" Ref="C?"  Part="1"
 AR Path="/5E7548ED/5F69C890" Ref="C13"  Part="1"
-F 0 "C13" H 4991 5196 50  0000 L CNN
-F 1 "?uF" H 4991 5105 50  0000 L CNN
-F 2 "Capacitor_SMD:C_0805_2012Metric" H 4900 5150 50  0001 C CNN
-F 3 "~" H 4900 5150 50  0001 C CNN
-	1    4900 5150
+F 0 "C13" H 5191 5446 50  0000 L CNN
+F 1 "68uF" H 5191 5355 50  0000 L CNN
+F 2 "Capacitor_SMD:C_1206_3216Metric" H 5100 5400 50  0001 C CNN
+F 3 "https://product.tdk.com/en/search/capacitor/ceramic/mlcc/info?part_no=C3216X5R1A686M160AC" H 5100 5400 50  0001 C CNN
+	1    5100 5400
 	-1   0    0    -1
 $EndComp
@@
 L LP3961EMP-5.0:LP3961EMP-5.0 IC3
 U 1 1 5F69DC3B
-P 5700 5250
-F 0 "IC3" H 6300 5518 50  0000 C CNN
-F 1 "LP3961EMP-5.0" H 6300 5425 50  0000 C CNN
-F 2 "LP3961EMP-5.0:SOT150P696X180-5N" H 6750 5350 50  0001 L CNN
-F 3 "" H 6750 5250 50  0001 L CNN
-F 4 "Fast Ultra Low Dropout Linear Regulators" H 6750 5150 50  0001 L CNN "Description"
-F 5 "" H 6750 5050 50  0001 L CNN "Height"
-F 6 "Texas Instruments" H 6750 4950 50  0001 L CNN "Manufacturer_Name"
-F 7 "LP3961EMP-5.0" H 6750 4850 50  0001 L CNN "Manufacturer_Part_Number"
-F 8 "LP3961EMP-5.0" H 6750 4750 50  0001 L CNN "Arrow Part Number"
-F 9 "https://www.arrow.com/en/products/lp3961emp-5.0/texas-instruments" H 6750 4650 50  0001 L CNN "Arrow Price/Stock"
-F 10 "926-LP3961EMP-50" H 6750 4550 50  0001 L CNN "Mouser Part Number"
-F 11 "https://www.mouser.com/Search/Refine.aspx?Keyword=926-LP3961EMP-50" H 6750 4450 50  0001 L CNN "Mouser Price/Stock"
-	1    5700 5250
+P 5850 5250
+F 0 "IC3" H 6350 5550 50  0000 C CNN
+F 1 "LP3961EMP-5.0" H 6350 5450 50  0000 C CNN
+F 2 "LP3961EMP-5.0:SOT150P696X180-5N" H 6900 5350 50  0001 L CNN
+F 3 "https://4donline.ihs.com/images/VipMasterIC/IC/NATL/NATLS08520/NATLS08520-1.pdf?hkey=EC6BD57738AE6E33B588C5F9AD3CEFA7" H 6900 5250 50  0001 L CNN
+F 4 "Fast Ultra Low Dropout Linear Regulators" H 6900 5150 50  0001 L CNN "Description"
+F 5 "" H 6900 5050 50  0001 L CNN "Height"
+F 6 "Texas Instruments" H 6900 4950 50  0001 L CNN "Manufacturer_Name"
+F 7 "LP3961EMP-5.0" H 6900 4850 50  0001 L CNN "Manufacturer_Part_Number"
+F 8 "LP3961EMP-5.0" H 6900 4750 50  0001 L CNN "Arrow Part Number"
+F 9 "https://www.arrow.com/en/products/lp3961emp-5.0/texas-instruments" H 6900 4650 50  0001 L CNN "Arrow Price/Stock"
+F 10 "926-LP3961EMP-50" H 6900 4550 50  0001 L CNN "Mouser Part Number"
+F 11 "https://www.mouser.com/Search/Refine.aspx?Keyword=926-LP3961EMP-50" H 6900 4450 50  0001 L CNN "Mouser Price/Stock"
+	1    5850 5250
 	1    0    0    -1
 $EndComp
@@
 L Device:R R?
 U 1 1 5F6A75BC
-P 5200 5450
+P 5450 5200
 AR Path="/5E755787/5F6A75BC" Ref="R?"  Part="1"
 AR Path="/5E755AC8/5D2551FF/5F6A75BC" Ref="R?"  Part="1"
-AR Path="/5E7548ED/5F6A75BC" Ref="R?"  Part="1"
-F 0 "R?" H 5270 5496 50  0000 L CNN
-F 1 "10k" H 5270 5405 50  0000 L CNN
-F 2 "Resistor_SMD:R_0805_2012Metric" V 5130 5450 50  0001 C CNN
-F 3 "~" H 5200 5450 50  0001 C CNN
-	1    5200 5450
-	1    0    0    -1
-$EndComp
+AR Path="/5E7548ED/5F6A75BC" Ref="R43"  Part="1"
+F 0 "R43" H 5520 5246 50  0000 L CNN
+F 1 "100k" H 5520 5155 50  0000 L CNN
+F 2 "Resistor_SMD:R_0805_2012Metric" V 5380 5200 50  0001 C CNN
+F 3 "~" H 5450 5200 50  0001 C CNN
+	1    5450 5200
+	1    0    0    -1
+$EndComp
+Wire Wire Line
+	5850 5400 5450 5400
+Wire Wire Line
+	5450 5400 5450 5350
+Wire Wire Line
+	6850 5500 7100 5500
+Wire Wire Line
+	6850 5300 6900 5300
+Wire Wire Line
+	6900 5300 6900 4800
+Wire Wire Line
+	6900 4800 7100 4800
+Wire Wire Line
+	5450 4800 5450 5050
+Wire Wire Line
+	7100 4800 7100 5100
+Wire Wire Line
+	7100 5400 7100 5500
+Connection ~ 7100 5500
+Wire Wire Line
+	7850 5750 7900 5750
+Wire Wire Line
+	7900 5750 7900 5950
+Wire Wire Line
+	8200 4650 8300 4650
+Wire Wire Line
+	8300 4650 8300 4800
+Wire Wire Line
+	7900 5950 7900 6100
+Wire Wire Line
+	7100 5500 7100 5750
+Wire Wire Line
+	5100 5550 5100 5750
+Wire Wire Line
+	5100 5750 5450 5750
+Wire Wire Line
+	6050 5750 6050 5850
+Wire Wire Line
+	5000 4800 5100 4800
+Connection ~ 5100 4800
+Wire Wire Line
+	5850 5250 5800 5250
+Wire Wire Line
+	5800 5250 5800 5150
+Wire Wire Line
+	5800 4800 5800 4850
+$Comp
+L Device:R R?
+U 1 1 5F535DE4
+P 5800 5000
+AR Path="/5E755787/5F535DE4" Ref="R?"  Part="1"
+AR Path="/5E755AC8/5D2551FF/5F535DE4" Ref="R?"  Part="1"
+AR Path="/5E7548ED/5F535DE4" Ref="R1"  Part="1"
+F 0 "R1" H 5870 5046 50  0000 L CNN
+F 1 "10k" H 5870 4955 50  0000 L CNN
+F 2 "Resistor_SMD:R_0805_2012Metric" V 5730 5000 50  0001 C CNN
+F 3 "~" H 5800 5000 50  0001 C CNN
+	1    5800 5000
+	-1   0    0    -1
+$EndComp
+Connection ~ 5450 4800
+Wire Wire Line
+	5450 4800 5800 4800
+Wire Wire Line
+	5100 4800 5300 4800
+Wire Wire Line
+	5100 4800 5100 5250
+Wire Wire Line
+	5300 4800 5300 5550
+Wire Wire Line
+	5300 5550 5850 5550
+Connection ~ 5300 4800
+Wire Wire Line
+	5300 4800 5450 4800
+Connection ~ 7100 4800
+Wire Wire Line
+	7100 4800 7200 4800
+Connection ~ 6050 5750
+Wire Wire Line
+	6050 5750 7100 5750
+Wire Wire Line
+	5450 5400 5450 5750
+Connection ~ 5450 5400
+Connection ~ 5450 5750
+Wire Wire Line
+	5450 5750 6050 5750
+Text Notes 4650 5950 0    50   ~ 0
+CIN ESR (mΩ) / CIN (μF) ≤ 1.5\nX7R or X5R Ceramic
+Text Notes 6350 5900 0    50   ~ 0
+0.2Ω ≤ COUT ESR ≤ 5Ω
+Text Notes 5950 4900 0    50   ~ 0
+See data sheet for\ncapacitor requirements
 $EndSCHEMATC
