File: Electronic Design/Core64 LB v0.4/Core64 LB v0.4 Power.sch (KiCad schematic (older format))
At the start: 29 parts, among them IC1 NCP176AMX330TCG, IC2 TPS7A0533PDBVR, IC3 LP3961EMP-5.0, J2 0.1\" 2-PIN, J3 Conn_01x08_Female, J8 S03B-PASK-2_LF__SN_, J9 JST-PH 2-PIN, Q22 BSS315PH6327XTSA1, SW1 JS102011SAQN, U6 Micro_LiPo_Charger

Commit message: Update schematic and XLS pin usage
Parts:
- H1, H2: footprint MountingHole:MountingHole_2.2mm_M2_Pad_Via -> MountingHole:MountingHole_3.2mm_M3_Pad_Via
Connections:
- net V_MON: no longer R51.2, R52.1
- new net VBAT_MON: R51.2, R52.1
Other:
- note added: "*** ALL CONFIGURATIONS REQUIRE CUTTING VIN-VUSB TRACE ON TEENSY ***"
- note added: "1S LIPO ONLY !!!"
- note added: "GND PAD 3.2 mm (.125 in) thru-hole for M3 or #4 screw"
- note added: "Mounting\n4x 0.1” holes"
- note added: "OPT: Open SJ to disable charging\nfrom Teensy USB. The USB port\non the charge manager will still work."
- note added: "SILKSCREEN: BAT. + BAT. -"
- note added: "SILKSCREEN: BAT. +/- pins"
- note added: "SILKSCREEN: GND"
- note added: "SILKSCREEN: LIPO CHARGER"
- note added: "SILKSCREEN: POWER"
- note removed: "*** ALL CONFIGURATIONS REQUIRED CUTTING VIN-VUSB TRACE ON TEENSY ***"
- note removed: "1S ONLY !!!"
- note removed: "OPT: Open SJ to\ndisable charging\nfrom Teensy USB."
- moved on the sheet: J9
Changed lines of the file:
@@
 	4100 5550 3850 5550
 Text GLabel 4100 5550 2    50   Output ~ 0
-V_MON
+VBAT_MON
 Text Notes 600  6850 0    118  ~ 0
 ALL SYSTEM STAR GROUNDING
@@
 F 0 "H2" H 1800 7250 50  0000 L CNN
 F 1 "GND PAD" H 1800 7157 50  0000 L CNN
-F 2 "MountingHole:MountingHole_2.2mm_M2_Pad_Via" H 1700 7200 50  0001 C CNN
+F 2 "MountingHole:MountingHole_3.2mm_M3_Pad_Via" H 1700 7200 50  0001 C CNN
 F 3 "~" H 1700 7200 50  0001 C CNN
 	1    1700 7200
@@
 F 0 "H1" H 1000 7250 50  0000 L CNN
 F 1 "GND PAD" H 800 7150 50  0000 L CNN
-F 2 "MountingHole:MountingHole_2.2mm_M2_Pad_Via" H 1200 7200 50  0001 C CNN
+F 2 "MountingHole:MountingHole_3.2mm_M3_Pad_Via" H 1200 7200 50  0001 C CNN
 F 3 "~" H 1200 7200 50  0001 C CNN
 	1    1200 7200
@@
 Text Notes 3500 2200 0    157  ~ 31
 7.5V MAX !!!
-Text Notes 3750 1900 0    50   ~ 0
-SILKSCREEN: +/- pins
+Text Notes 2200 2150 0    50   ~ 0
+SILKSCREEN: BAT. +/- pins
 Text GLabel 4800 7450 1    50   Input ~ 0
 RPP
@@
 P-FET
 Text Notes 750  4100 0    157  ~ 31
-*** ALL CONFIGURATIONS REQUIRED CUTTING VIN-VUSB TRACE ON TEENSY ***
+*** ALL CONFIGURATIONS REQUIRE CUTTING VIN-VUSB TRACE ON TEENSY ***
 Text GLabel 5400 7450 1    50   Output ~ 0
 V_MON
-Text Notes 8900 2200 0    157  ~ 31
-1S ONLY !!!
+Text Notes 8250 2150 0    157  ~ 31
+1S LIPO ONLY !!!
 Text Notes 6800 3050 0    50   ~ 0
 ALTERNATE CONNECTOR - JST-PH 2-PIN SMT\nAdafruit 1769 Right Angle Battery Cable Socket\nJST S2B-PH-SM4-TB(LF)(SN), Digi-Key 455-1749-1-ND
@@
 L Connector:Conn_01x02_Male J9
 U 1 1 5F5849A5
-P 7450 3350
-F 0 "J9" H 7450 3450 50  0000 C CNN
-F 1 "JST-PH 2-PIN" H 7500 3150 50  0000 C CNN
-F 2 "Connector_JST:JST_PH_S2B-PH-SM4-TB_1x02-1MP_P2.00mm_Horizontal" H 7450 3350 50  0001 C CNN
-F 3 "~" H 7450 3350 50  0001 C CNN
-	1    7450 3350
+P 7950 3350
+F 0 "J9" H 7950 3450 50  0000 C CNN
+F 1 "JST-PH 2-PIN" H 8000 3150 50  0000 C CNN
+F 2 "Connector_JST:JST_PH_S2B-PH-SM4-TB_1x02-1MP_P2.00mm_Horizontal" H 7950 3350 50  0001 C CNN
+F 3 "~" H 7950 3350 50  0001 C CNN
+	1    7950 3350
 	1    0    0    -1
 $EndComp
@@
 L power:+BATT #PWR0156
 U 1 1 5F586B8B
-P 8200 3350
+P 8700 3350
 AR Path="/5E7548ED/5F586B8B" Ref="#PWR0156"  Part="1"
 AR Path="/5E755AC8/5D254AE8/5F586B8B" Ref="#PWR?"  Part="1"
-F 0 "#PWR0156" H 8200 3200 50  0001 C CNN
-F 1 "+BATT" H 8215 3523 50  0000 C CNN
-F 2 "" H 8200 3350 50  0001 C CNN
-F 3 "" H 8200 3350 50  0001 C CNN
-	1    8200 3350
+F 0 "#PWR0156" H 8700 3200 50  0001 C CNN
+F 1 "+BATT" H 8715 3523 50  0000 C CNN
+F 2 "" H 8700 3350 50  0001 C CNN
+F 3 "" H 8700 3350 50  0001 C CNN
+	1    8700 3350
 	1    0    0    -1
 $EndComp
@@
 L power:-BATT #PWR0159
 U 1 1 5F586B91
-P 8200 3450
+P 8700 3450
 AR Path="/5E7548ED/5F586B91" Ref="#PWR0159"  Part="1"
 AR Path="/5E755AC8/5D254AE8/5F586B91" Ref="#PWR?"  Part="1"
-F 0 "#PWR0159" H 8200 3300 50  0001 C CNN
-F 1 "-BATT" H 8215 3623 50  0000 C CNN
-F 2 "" H 8200 3450 50  0001 C CNN
-F 3 "" H 8200 3450 50  0001 C CNN
-	1    8200 3450
+F 0 "#PWR0159" H 8700 3300 50  0001 C CNN
+F 1 "-BATT" H 8715 3623 50  0000 C CNN
+F 2 "" H 8700 3450 50  0001 C CNN
+F 3 "" H 8700 3450 50  0001 C CNN
+	1    8700 3450
 	-1   0    0    1
 $EndComp
 Wire Wire Line
-	7650 3350 8200 3350
-Wire Wire Line
-	7650 3450 8200 3450
+	8150 3350 8700 3350
+Wire Wire Line
+	8150 3450 8700 3450
 Text Notes 1850 6550 0    50   ~ 0
 OPTIONAL FET PROTECT:\n1) .1uF Cap. on left\n2) 100k Res. on bottom\n3) 10V Zener on right
@@
 SILKSCREEN: +/- pins
 Text Notes 5300 2450 0    50   ~ 0
-TWO OPTIONS\n\n1) 1S LiPo + Charger (most convenient)\n     A) Choose a 1S Lipo with built-in cell over/under voltage protection. Recommended \n     B) Choose a charger. The logic board is designed to accept this one: https://www.adafruit.com/product/1904\n     C) 4-pin header to connector charger to the logic board. Or solder direct to logic board.\n\n2) 1S LiPo only (flexible, choose your own connector)\n     A) Choose a 1S LiPo with protection circuit, up to 50 x 55 x 12mm\n\nINSTRUCTIONS\nA) Remove the 4x “AAA” battery pack. Reuse the connector if you want to.\nB) Install the charge manager if you want to.\nC) Install the 1S LiPo with double-sided tape.\n\n* The LiPo charger 5V pin is also connected to the Teensy USB port.\n* Connecting a USB cable to the Teensy will power the board, charge the battery\n* and connect to the serial port of the Teensy. Connecting a USB cable to the LiPO\n* charger will ONLY charge the battery and power the logic board.
+TWO OPTIONS\n\n1) 1S LiPo + Charger (most convenient)\n     A) Choose a 1S Lipo with built-in cell over/under voltage protection. Recommended \n     B) Choose a charger. The logic board is designed to accept this one: https://www.adafruit.com/product/1904\n     C) 4-pin header to connector charger to the logic board. Or solder direct to logic board.\n\n2) 1S LiPo only (flexible, choose your own connector)\n     A) Choose a 1S LiPo with protection circuit, up to 50 x 55 x 12mm\n\nINSTRUCTIONS\nA) Remove the 4x “AAA” battery pack.\nB) Install the charge manager (optional).\nC) Install the 1S LiPo with double-sided tape.\n\n* The LiPo charger 5V pin is also connected to the Teensy USB port.\n* Connecting a USB cable to the Teensy will power the board, charge the battery\n* and connect to the serial port of the Teensy. Connecting a USB cable to the LiPO\n* charger will ONLY charge the battery and power the logic board.
 Wire Wire Line
 	4500 7650 4650 7650
@@
 $EndComp
 Text Notes 6050 3700 0    50   ~ 0
-OPT: Open SJ to\ndisable charging\nfrom Teensy USB.
+OPT: Open SJ to disable charging\nfrom Teensy USB. The USB port\non the charge manager will still work.
 Wire Wire Line
 	5900 3300 6100 3300
@@
 Wire Wire Line
 	9550 6000 9850 6000
-Text Notes 10000 6150 0    50   ~ 0
+Text Notes 9900 6450 0    118  ~ 24
 Must\nSelect\nOne
 Text GLabel 8200 4650 0    50   Input ~ 0
@@
 Text Notes 5950 4900 0    50   ~ 0
 See data sheet for\ncapacitor requirements
+Text Notes 750  7000 0    50   ~ 0
+GND PAD 3.2 mm (.125 in) thru-hole for M3 or #4 screw
+Text Notes 2200 7150 0    50   ~ 0
+SILKSCREEN: GND
+Text Notes 5300 2650 0    50   ~ 0
+SILKSCREEN: LIPO CHARGER
+Text Notes 8400 2700 0    50   ~ 0
+SILKSCREEN: BAT. + BAT. -
+Text Notes 4850 7000 0    50   ~ 0
+SILKSCREEN: POWER
+Text Notes 6000 3100 0    50   ~ 0
+Mounting\n4x 0.1” holes
 $EndSCHEMATC

Commit message: Update schematic
Parts:
- added J18: 5V0 Cur. Mon., Connector_PinSocket_2.54mm:PinSocket_1x02_P2.54mm_Vertical, symbol Connector_Generic:Conn_01x02
- added J19: 3V3 Cur. Mon., Connector_PinSocket_2.54mm:PinSocket_1x02_P2.54mm_Vertical, symbol Connector_Generic:Conn_01x02
Connections:
- net V_MON is gone; now on net VBAT_MON: J3.7 (Pin_7)
- net 3V3: now also J19.1 (Pin_1), J19.2 (Pin_2)
- net 5V0: now also J18.1 (Pin_1), J18.2 (Pin_2)
Other:
- note added: "OPTIONAL USB BYPASS:\nAs shipped, power switch\nin OFF position connects\nto USB power through\nthe Teensy.\nOPTIONAL:\nCut SJ if you want the \nOFF position to not\nbe powered from\nTeensy USB connector."
- note removed: "OPTIONAL USB BYPASS:\nAs shipped, switch in\nOFF position connects\nto USB power through\nthe Teensy.\nOPTIONAL:\nCut SJ if you want the \nOFF position to not\nbe powered from\nTeensy USB connector."
- moved on the sheet: C12, C2, IC2, JP9

Commit message: Update footprint mounting holes TFT, LED array, battery packs, lipo charger, arrange components to fit on the board
Parts:
- removed J2: 0.1\" 2-PIN, Connector_PinSocket_2.54mm:PinSocket_1x02_P2.54mm_Vertical_SMD_Pin1Left, symbol Connector:Conn_01x02_Male
- removed J9: JST-PH 2-PIN, Connector_JST:JST_PH_S2B-PH-SM4-TB_1x02-1MP_P2.00mm_Horizontal, symbol Connector:Conn_01x02_Male
- C7: footprint Capacitor_SMD:CP_Elec_10x10 -> Capacitor_SMD:CP_Elec_6.3x7.7
- JP8: footprint Jumper:SolderJumper-2_P1.3mm_Bridged_Pad1.0x1.5mm -> Jumper:SolderJumper-2_P1.3mm_Bridged_RoundedPad1.0x1.5mm
Connections:
- net -BATT: now also IC1.3 (GND_1)
Other:
- note added: "1) Remove the 4x “AAA” battery pack. You can leave \n\n2) Purchase and install a LiPo charge manager.\n a) The logic board is designed to accept this one: https://www.adafruit.com/product/1904.\n b) Solder the the charge manager directly to the board without headers to keep a low profile to allow the stylus to fit.\n\n3) Purchase and install a 1S LiPo using double-sided tape. \n a) Choose a 1S Li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"
- note removed: "ALTERNATE CONNECTOR - JST-PH 2-PIN SMT\nAdafruit 1769 Right Angle Battery Cable Socket\nJST S2B-PH-SM4-TB(LF)(SN), Digi-Key 455-1749-1-ND"
- note removed: "ALTERNATE CONNECTOR\nGeneric 2-pin header 0.1”"
- note removed: "HIGH POWER SYSTEM GROUND"
- note removed: "TWO OPTIONS\n\n1) 1S LiPo + Charger (most convenient)\n A) Choose a 1S Lipo with built-in cell over/under voltage protection. Recommended \n B) Choose a charger. The logic board is designed to accept this one: https://www.adafruit.com/product/1904\n C) 4-pin header to connector charger to the logic board. Or solder direct to logic board.\n\n2) 1S LiPo only (flexible, choose your own connector)\n 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"
Changed lines of the file:
@@
 SOURCE 2 “OFF (USB)”\n  USB 5V supplied through Teensy 3.2 \n  With the VIN-VUSB trace cut on the back of the Teensy, the TEENSY_5VUSB\n  is routed directly from the USB Port, to the VUSB pin on the back \n  of the Teensy, over to one side of the SPDT switch. In this position\n  the VUSB goes back to the Teensy through the 5V regulator.
-$Comp
-L Connector:Conn_01x02_Male J2
-U 1 1 5E78F60B
-P 9350 3350
-AR Path="/5E7548ED/5E78F60B" Ref="J2"  Part="1"
-AR Path="/5E755AC8/5D254AE8/5E78F60B" Ref="J?"  Part="1"
-F 0 "J2" H 9350 3450 50  0000 C CNN
-F 1 "0.1\" 2-PIN" H 9350 3150 50  0000 C CNN
-F 2 "Connector_PinSocket_2.54mm:PinSocket_1x02_P2.54mm_Vertical_SMD_Pin1Left" H 9350 3350 50  0001 C CNN
-F 3 "~" H 9350 3350 50  0001 C CNN
-	1    9350 3350
-	1    0    0    -1
-$EndComp
 $Comp
 L power:+BATT #PWR0105
@@
 	-1   0    0    1
 $EndComp
-$Comp
-L power:+BATT #PWR0107
-U 1 1 5E795118
-P 10100 3350
-AR Path="/5E7548ED/5E795118" Ref="#PWR0107"  Part="1"
-AR Path="/5E755AC8/5D254AE8/5E795118" Ref="#PWR?"  Part="1"
-F 0 "#PWR0107" H 10100 3200 50  0001 C CNN
-F 1 "+BATT" H 10115 3523 50  0000 C CNN
-F 2 "" H 10100 3350 50  0001 C CNN
-F 3 "" H 10100 3350 50  0001 C CNN
-	1    10100 3350
-	1    0    0    -1
-$EndComp
-$Comp
-L power:-BATT #PWR0108
-U 1 1 5E79511E
-P 10100 3450
-AR Path="/5E7548ED/5E79511E" Ref="#PWR0108"  Part="1"
-AR Path="/5E755AC8/5D254AE8/5E79511E" Ref="#PWR?"  Part="1"
-F 0 "#PWR0108" H 10100 3300 50  0001 C CNN
-F 1 "-BATT" H 10115 3623 50  0000 C CNN
-F 2 "" H 10100 3450 50  0001 C CNN
-F 3 "" H 10100 3450 50  0001 C CNN
-	1    10100 3450
-	-1   0    0    1
-$EndComp
 Text Notes 650  1000 0    50   ~ 0
 TWO POWER INPUT SOURCES SELECTED BY SPDT SWITCH
@@
 Wire Wire Line
 	1550 2250 2150 2250
-Wire Wire Line
-	9550 3350 10100 3350
-Wire Wire Line
-	9550 3450 10100 3450
 Wire Notes Line style solid
 	600  850  5000 850
@@
 	10350 850  5200 850
 Connection ~ 3850 5250
-Text Notes 9300 6550 2    50   ~ 0
-HIGH POWER SYSTEM GROUND
 Text Notes 5800 4550 0    50   ~ 0
 LED ARRAY, TEENSY VIN
@@
 Text Notes 600  6850 0    118  ~ 0
 ALL SYSTEM STAR GROUNDING
-Text Notes 9200 2950 0    50   ~ 0
-ALTERNATE CONNECTOR\nGeneric 2-pin header 0.1”
 Wire Wire Line
 	1550 2050 2150 2050
@@
 	1    0    0    -1
 $EndComp
-Text Notes 5550 6150 0    50   ~ 0
-HIGH POWER SYSTEM GROUND
 Connection ~ 3850 5550
 Text Notes 3500 2200 0    157  ~ 31
@@
 Text GLabel 5400 7450 1    50   Output ~ 0
 VBAT_MON
-Text Notes 8250 2150 0    157  ~ 31
+Text Notes 7600 3150 0    157  ~ 31
 1S LIPO ONLY !!!
-Text Notes 6800 3050 0    50   ~ 0
-ALTERNATE CONNECTOR - JST-PH 2-PIN SMT\nAdafruit 1769 Right Angle Battery Cable Socket\nJST S2B-PH-SM4-TB(LF)(SN), Digi-Key 455-1749-1-ND
 $Comp
 L CORE_64_LIBRARY:Micro_LiPo_Charger U6
@@
 Wire Wire Line
 	5600 3400 5600 3450
-$Comp
-L Connector:Conn_01x02_Male J9
-U 1 1 5F5849A5
-P 7950 3350
-F 0 "J9" H 7950 3450 50  0000 C CNN
-F 1 "JST-PH 2-PIN" H 8000 3150 50  0000 C CNN
-F 2 "Connector_JST:JST_PH_S2B-PH-SM4-TB_1x02-1MP_P2.00mm_Horizontal" H 7950 3350 50  0001 C CNN
-F 3 "~" H 7950 3350 50  0001 C CNN
-	1    7950 3350
-	1    0    0    -1
-$EndComp
-$Comp
-L power:+BATT #PWR0156
-U 1 1 5F586B8B
-P 8700 3350
-AR Path="/5E7548ED/5F586B8B" Ref="#PWR0156"  Part="1"
-AR Path="/5E755AC8/5D254AE8/5F586B8B" Ref="#PWR?"  Part="1"
-F 0 "#PWR0156" H 8700 3200 50  0001 C CNN
-F 1 "+BATT" H 8715 3523 50  0000 C CNN
-F 2 "" H 8700 3350 50  0001 C CNN
-F 3 "" H 8700 3350 50  0001 C CNN
-	1    8700 3350
-	1    0    0    -1
-$EndComp
-$Comp
-L power:-BATT #PWR0159
-U 1 1 5F586B91
-P 8700 3450
-AR Path="/5E7548ED/5F586B91" Ref="#PWR0159"  Part="1"
-AR Path="/5E755AC8/5D254AE8/5F586B91" Ref="#PWR?"  Part="1"
-F 0 "#PWR0159" H 8700 3300 50  0001 C CNN
-F 1 "-BATT" H 8715 3623 50  0000 C CNN
-F 2 "" H 8700 3450 50  0001 C CNN
-F 3 "" H 8700 3450 50  0001 C CNN
-	1    8700 3450
-	-1   0    0    1
-$EndComp
-Wire Wire Line
-	8150 3350 8700 3350
-Wire Wire Line
-	8150 3450 8700 3450
 Text Notes 1850 6550 0    50   ~ 0
 OPTIONAL FET PROTECT:\n1) .1uF Cap. on left\n2) 100k Res. on bottom\n3) 10V Zener on right
@@
 SILKSCREEN: +/- pins
 Text Notes 5300 2450 0    50   ~ 0
-TWO OPTIONS\n\n1) 1S LiPo + Charger (most convenient)\n     A) Choose a 1S Lipo with built-in cell over/under voltage protection. Recommended \n     B) Choose a charger. The logic board is designed to accept this one: https://www.adafruit.com/product/1904\n     C) 4-pin header to connector charger to the logic board. Or solder direct to logic board.\n\n2) 1S LiPo only (flexible, choose your own connector)\n     A) Choose a 1S LiPo with protection circuit, up to 50 x 55 x 12mm\n\nINSTRUCTIONS\nA) Remove the 4x “AAA” battery pack.\nB) Install the charge manager (optional).\nC) Install the 1S LiPo with double-sided tape.\n\n* The LiPo charger 5V pin is also connected to the Teensy USB port.\n* Connecting a USB cable to the Teensy will power the board, charge the battery\n* and connect to the serial port of the Teensy. Connecting a USB cable to the LiPO\n* charger will ONLY charge the battery and power the logic board.
+1) Remove the 4x “AAA” battery pack. You can leave \n\n2) Purchase and install a LiPo charge manager.\n     a) The logic board is designed to accept this one: https://www.adafruit.com/product/1904.\n     b) Solder the the charge manager directly to the board without headers to keep a low profile to allow the stylus to fit.\n\n3) Purchase and install a 1S LiPo using double-sided tape. \n     a) Choose a 1S Lipo with built-in cell over/under voltage protection. Recommended:\n          2500mAh https://www.adafruit.com/product/328   1.8” x 2.4” x 0.26” (47mm x 61mm x 6.7mm)\n          2000mAh https://www.adafruit.com/product/2011  2.4” x 1.4” x 0.3” (60mm x 36mm x 7mm)\n          1200mAh https://www.adafruit.com/product/258    1.3” x 2.4” x 0.2” (34mm x 62mm x 5mm)\n     b) The LiPo can be up to 50 x 65 x 15mm. A maximum \n     a) Make sure no part of the LiPo foil pouch can short-out adjacent pins or pads in the area.\n     b) Insulate it with Kapton tape or similar.\n\n* The LiPo charger 5V pin is also connected to the Teensy USB port.\n* Connecting a USB cable to the Teensy will power the board, charge the battery and connect to the serial port of the\n   Teensy. If you do NOT want the board to be powered from the USB port of the charger, cut the 5V solder jumper.\n* Connecting a USB cable to the LiPO charger will ONLY charge the battery and power the logic board.
 Wire Wire Line
 	4500 7650 4650 7650
@@
 F 0 "JP8" H 6250 3200 50  0000 C CNN
 F 1 "Teensy_Charge_Enable" H 6050 3400 50  0000 C CNN
-F 2 "Jumper:SolderJumper-2_P1.3mm_Bridged_Pad1.0x1.5mm" H 6250 3300 50  0001 C CNN
+F 2 "Jumper:SolderJumper-2_P1.3mm_Bridged_RoundedPad1.0x1.5mm" H 6250 3300 50  0001 C CNN
 F 3 "~" H 6250 3300 50  0001 C CNN
 	1    6250 3300
@@
 	1    0    0    -1
 $EndComp
-Text Notes 8250 5650 0    50   ~ 0
+Text Notes 8350 5700 0    50   ~ 0
 Preferred, TINY
-Text Notes 8350 4650 0    50   ~ 0
+Text Notes 8350 4700 0    50   ~ 0
 Alternate, larger
 $Comp
@@
 	1    0    0    -1
 $EndComp
-Text Notes 8100 5400 0    50   ~ 0
-HIGH POWER SYSTEM GROUND
 Wire Wire Line
 	9250 6100 9300 6100
@@
 F 0 "C7" H 7191 5296 50  0000 L CNN
 F 1 "470uF" H 7191 5205 50  0000 L CNN
-F 2 "Capacitor_SMD:CP_Elec_10x10" H 7100 5250 50  0001 C CNN
+F 2 "Capacitor_SMD:CP_Elec_6.3x7.7" H 7100 5250 50  0001 C CNN
 F 3 "" H 7100 5250 50  0001 C CNN
 F 4 "565-EMHL100ARA471MHA0GCT-ND" H 7100 5250 50  0001 C CNN "Digikey"
@@
 Text Notes 2200 7150 0    50   ~ 0
 SILKSCREEN: GND
-Text Notes 5300 2650 0    50   ~ 0
+Text Notes 6450 2850 0    50   ~ 0
 SILKSCREEN: LIPO CHARGER
-Text Notes 8400 2700 0    50   ~ 0
+Text Notes 8150 3350 0    50   ~ 0
 SILKSCREEN: BAT. + BAT. -
 Text Notes 4750 6950 0    50   ~ 0
@@
 Text Notes 6000 3100 0    50   ~ 0
 Mounting\n4x 0.1” holes
-Text Label 2250 7450 0    50   ~ 0
-GND
 $Comp
 L Connector_Generic:Conn_01x02 J18
@@
 Connection ~ 10000 5550
 Connection ~ 10100 5550
+Wire Wire Line
+	9250 6200 9300 6200
+Wire Wire Line
+	9300 6200 9300 6450
+Wire Wire Line
+	9300 6450 8050 6450
+Wire Wire Line
+	8050 6450 8050 6350
+Wire Wire Line
+	8050 6350 7900 6350
 $EndSCHEMATC
