File: Electronic Design/Core64 CB v0.4-NP/Core64 CB v0.4-NP.sch (KiCad schematic (older format))
At the start: 16 parts, among them J1 TSM-116-03-T-SV‎, J2 TSM-116-03-T-SV‎, U1 SI7210-B-01, U2 SI7210-B-02, U3 SI7210-B-03, U4 SI7210-B-04, U5 LTR-329ALS-01, X1 SAO_conn_SFH11-NBPC-D03-ST-BK

Commit message: Update Simple Add Ons #2 on all schematics PCBs
Other:
- note added: "SILKSCREEN FRONT AND BACK: \nSAO#2, GNDD, 3V3, SDA,SCL\nGPIO1, GPIO2"
- note added: "SIMPLE ADD ONS see:\nhttps://hackaday.io/project/175182-simple-add-ons-sao"
- note added: "[OPTIONAL] SAO #2 EXPANSION"
- note removed: "SILKSCREEN FRONT AND BACK: \nSAO, GNDD, 3V3, SDA,SCL\nGPIO1, GPIO2"
- note removed: "[OPTIONAL] SAO EXPANSION"
Changed lines of the file:
@@
 	6700 2350 6950 2350
 Text Notes 8850 1200 0    50   ~ 0
-SILKSCREEN FRONT AND BACK: \nSAO, GNDD, 3V3, SDA,SCL\nGPIO1, GPIO2
+SILKSCREEN FRONT AND BACK: \nSAO#2, GNDD, 3V3, SDA,SCL\nGPIO1, GPIO2
 $Comp
 L Device:C C5
@@
 Text Notes 600  700  0    100  ~ 0
 CORE MATRIX
-Text Notes 7950 800  0    100  ~ 0
-[OPTIONAL] SAO EXPANSION
+Text Notes 7900 700  0    100  ~ 0
+[OPTIONAL] SAO #2 EXPANSION
 Text Notes 1600 3200 0    50   ~ 0
 SILKSCREEN: 0x30
@@
 Text Notes 5600 7250 0    50   ~ 0
 NEON\nPIXELS\nEDITION
+Text Notes 7950 900  0    50   ~ 0
+SIMPLE ADD ONS see:\nhttps://hackaday.io/project/175182-simple-add-ons-sao
 $EndSCHEMATC
