File: Electronic Design/Core64 LM v0.1/Core64 LM v0.1 Expansion.sch (KiCad schematic (older format))
At the start: 7 parts

Commit message: Finish layout, revise notes
Parts:
- JP3: value SolderJumper_2_Open -> Teensy_Charge_Enable
Other:
- note added: "* Do not connect AAAs to a LiPo charger! You will destroy it.\n\n1) Remove the 4x “AAA” battery pack.\n\n2) Purchase and install a LiPo charge manager.\n a) The logic board is designed to accept this one: https://www.adafruit.com/product/1904 (Micro USB) or 4410 (USB C).\n b) Solder the the charge manager directly to the board without headers to keep a low profile.\n\n3) Purchase and install a 1S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"
- note added: "0.96” (128x64)\nI2C 4-pins, ADDRESS: 0x3C (60 decimal)\nAlternate is 0x3D, not 0x7A or 0x78 (wrong 8-bit)!\nMust choose power polarity by soldering SJs."
- note added: "1S LIPO ONLY !!!"
- note added: "ALTERNATE 1S LIPO BATTERY - USER SUPPLIED"
- note added: "Mounting\n4x 0.1” holes"
- note added: "SILKSCREEN: +/- pins"
- note added: "SILKSCREEN: BAT. + BAT. -"
- note added: "SILKSCREEN: LIPO CHARGER"
- note removed: "0.96” (128x64)\nI2C 4-pins, ADDRESS: 0x3C (60 decimal)\nAlternate is 0x3D, not 0x7A or 0x78 (wrong 8-bit)!\nMust choose power polarity by soldering SJS."
- note removed: "CLOSE SOLDER JUMPER TO\nENABLE CHARGING OF BATTERY\nWHEN THE MICROCONTROLLER IS\nPOWERED BY USB/PROGRAMMING\nCONNECTION."
- moved on the sheet: JP1, JP2, JP3, XLM1, XLM2, XLM3, XLM4

Commit message: Tweak layout and silk screen
Other:
- note added: "SILKSCREEN:\n1S ONLY\nADAFRUIT #1904 MICRO USB\nADAFRUIT #4410 USB C"
- note removed: "All non-polarized capacitors are X7R or X5R ceramic unless otherwise noted."
- note removed: "SILKSCREEN:\n1S ONLY\nADAFRUIT #1904 MICROUSB\nADAFRUIT #4410 TYPE C USB"
Changed lines of the file:
@@
 encoding utf-8
 Sheet 2 2
-Title "Core 64 LED Matrix - Expansion"
-Date "2021-02-12"
+Title "Core64 LM (LED MATRIX)"
+Date "2021-02-17"
 Rev "0.1"
-Comp "www.Core64.io"
-Comment1 "Work in progress"
-Comment2 "Andy Geppert"
+Comp "Concept and design by Andy Geppert @ www.MachineIdeas.com"
+Comment1 "Visit www.Core64.io for information on assembly and optional features."
+Comment2 "*** Work in progress ***"
 Comment3 ""
-Comment4 ""
+Comment4 "All capacitors ceramic X7R unless otherwise noted."
 $EndDescr
 Text GLabel 2450 1850 0    50   BiDi ~ 0
@@
 Text Notes 900  2900 0    50   ~ 0
 SILKSCREEN: 3V3 ONLY, 3V3/GNDD sides of jumpers,\nI2C OLED and pin names
-Text Notes 6300 6750 0    50   ~ 0
-All non-polarized capacitors are X7R or X5R ceramic unless otherwise noted.
 Connection ~ 1650 1900
 Wire Wire Line
@@
 	6700 4600 7300 4600
 Text Notes 4300 4800 0    50   ~ 0
-SILKSCREEN:\n1S ONLY\nADAFRUIT #1904 MICROUSB\nADAFRUIT #4410 TYPE C USB
+SILKSCREEN:\n1S ONLY\nADAFRUIT #1904 MICRO USB\nADAFRUIT #4410 USB C
 $Comp
 L Jumper:SolderJumper_2_Open JP3
@@
 Mounting\n4x 0.1” holes
 Text Notes 4300 3900 0    50   ~ 0
-* Do not connect AAAs to a LiPo charger! You will destroy it.\n\n1) Remove the 4x “AAA” battery pack.\n\n2) Purchase and install a LiPo charge manager.\n     a) The logic board is designed to accept this one: https://www.adafruit.com/product/1904 (Micro USB) or 4410 (USB C).\n     b) Solder the the charge manager directly to the board without headers to keep a low profile.\n\n3) Purchase and install a 1S LiPo using double-sided tape. \n     a) Choose a 1S Lipo with built-in cell over/under voltage protection. Recommended:\n          2500mAh https://www.adafruit.com/product/328   1.8” x 2.4” x 0.26” (47mm x 61mm x 6.7mm)\n          2000mAh https://www.adafruit.com/product/2011  2.4” x 1.4” x 0.3” (60mm x 36mm x 7mm)\n          1200mAh https://www.adafruit.com/product/258    1.3” x 2.4” x 0.2” (34mm x 62mm x 5mm)\n     b) The LiPo can be up to 50 x 65 x 15mm.\n     a) Make sure no part of the LiPo foil pouch can short-out adjacent pins or pads in the area. Insulate it with Kapton tape or similar.\n\n\nConfiguration of the Teensy_Charge_Enable Solder Jumper (SJ):\nA) DEFAULT SJ OPEN:\n       If you do NOT want the system to be powered from the USB port of the charger, leave the Teensy_Charge_Enable SJ open.\n       Connecting a USB cable to the LiPo charger will ONLY charge the battery and power the system when the power switch is ON (up position).\n       Connecting a USB cable to the Teensy will NOT charge the battery.\n\nB) OPTIONAL SJ CLOSED:\n       The LiPo charger 5V pin (Lipo Charger USB port) may be connected to the Teensy USB port through TEENSY_VUSB. Close the SJ to connect them.\n       Connecting a USB cable to the LiPo charger will charge the battery and power the system \n       Connecting a USB cable to the Teensy will power the Core64 board, charge the battery and connect to the serial port of the Teensy.\n
+* Do not connect AAAs to a LiPo charger! You will destroy it.\n\n1) Remove the 4x “AAA” battery pack.\n\n2) Purchase and install a LiPo charge manager.\n     a) The logic board is designed to accept this one: https://www.adafruit.com/product/1904 (Micro USB) or 4410 (USB C).\n     b) Solder the the charge manager directly to the board without headers to keep a low profile.\n\n3) Purchase and install a 1S LiPo using double-sided tape. \n     a) Choose a 1S Lipo with built-in cell over/under voltage protection. Recommended:\n          2500mAh https://www.adafruit.com/product/328   1.8” x 2.4” x 0.26” (47mm x 61mm x 6.7mm)\n          2000mAh https://www.adafruit.com/product/2011  2.4” x 1.4” x 0.3” (60mm x 36mm x 7mm)\n          1200mAh https://www.adafruit.com/product/258    1.3” x 2.4” x 0.2” (34mm x 62mm x 5mm)\n     b) Make sure no part of the LiPo foil pouch can short-out adjacent pins or pads in the area. Insulate it with Kapton tape or similar.\n\n\nConfiguration of the Teensy_Charge_Enable Solder Jumper (SJ):\nA) DEFAULT SJ OPEN:\n       If you do NOT want the system to be powered from the USB port of the charger, leave the Teensy_Charge_Enable SJ open.\n       Connecting a USB cable to the LiPo charger will ONLY charge the battery and power the system when the power switch is ON (up position).\n       Connecting a USB cable to the Teensy will NOT charge the battery.\n\nB) OPTIONAL SJ CLOSED:\n       The LiPo charger 5V pin (Lipo Charger USB port) may be connected to the Teensy USB port through TEENSY_VUSB. Close the SJ to connect them.\n       Connecting a USB cable to the LiPo charger will charge the battery and power the system \n       Connecting a USB cable to the Teensy will power the Core64 board, charge the battery and connect to the serial port of the Teensy.\n
 $EndSCHEMATC

Commit message: Create BOM and CPL
Other:
- note added: "1S LIPO ONLY !!!\n7.5V ABSOLUTE MAXIMUM !!!"
- note removed: "1S LIPO ONLY !!!"
Changed lines of the file:
@@
 Sheet 2 2
 Title "Core64 LM (LED MATRIX)"
-Date "2021-02-17"
+Date "2021-02-18"
 Rev "0.1"
 Comp "Concept and design by Andy Geppert @ www.MachineIdeas.com"
 Comment1 "Visit www.Core64.io for information on assembly and optional features."
-Comment2 "*** Work in progress ***"
+Comment2 "*** As released 2021-02-18 ***"
 Comment3 ""
 Comment4 "All capacitors ceramic X7R unless otherwise noted."
@@
 Text Notes 4300 1300 0    118  ~ 0
 ALTERNATE 1S LIPO BATTERY - USER SUPPLIED
-Text Notes 5800 5800 0    157  ~ 31
-1S LIPO ONLY !!!
+Text Notes 5000 6100 0    157  ~ 31
+1S LIPO ONLY !!!\n7.5V ABSOLUTE MAXIMUM !!!
 Text Notes 5500 5350 0    50   ~ 0
 SILKSCREEN: +/- pins
