File: Electronic Design/Core64 LM v0.1/Core64 LM v0.1.kicad_pcb (KiCad board)
At the start: 2 copper layers, 85 x 85 mm, 78 parts, among them J1 Digi-Key 77311-420-36LF-ND, J2 Digi-Key 77311-420-36LF-ND, J3 Conn_01x03_Male

Commit message: Add optional LiPo charger, QWIIC, OLED I2C to LED Matrix, change to start with V0.1
Parts:
- removed ? (x2): , 
- removed J3: Conn_01x03_Male, Connector_PinHeader_2.54mm:PinHeader_1x03_P2.54mm_Vertical
- added JP1: SolderJumper_3_Open, Jumper:SolderJumper-3_P1.3mm_Open_Pad1.0x1.5mm_NumberLabels, F.Cu at (-8.26, 30.5)
- added JP2: SolderJumper_3_Open, Jumper:SolderJumper-3_P1.3mm_Open_Pad1.0x1.5mm_NumberLabels, F.Cu at (-8.26, 34.0)
- added JP3: SolderJumper_2_Open, Jumper:SolderJumper-2_P1.3mm_Open_Pad1.0x1.5mm, B.Cu at (-39.0, 24.1)
- added XLM1: Micro_LiPo_Charger, Core_Memory_8x8_Array:Micro_LiPo_Charger_CornerSMD, B.Cu at (22.2, -31.8)
- added XLM2: Conn_01x04_Male, Connector_PinHeader_2.54mm:PinHeader_1x04_P2.54mm_Vertical, F.Cu at (0.00, 39.0)
- added XLM3: QWIIC, Connector_JST:JST_SH_SM04B-SRSS-TB_1x04-1MP_P1.00mm_Horizontal, F.Cu at (-19.7, 36.8)
- added XLM4: Conn_01x03_Male, Connector_PinHeader_2.54mm:PinHeader_1x03_P2.54mm_Vertical, F.Cu at (-17.2, -30.5)
- J1, J2: value Digi-Key 77311-420-36LF-ND -> PASS THROUGH BOARD; footprint Connector_PinHeader_2.54mm:PinHeader_1x18_P2.54mm_Vertical_SMD_and_TH_Pin1Right -> Connector_PinHeader_2.54mm:PinHeader_1x20_P2.54mm_Vertical_SMD_and_TH_Pin1Right
- moved L1 13.4 mm to (-10.8, -36.8)
Connections:
- J1 pad 11: Net-(J1-Pad11) -> I2C_CLOCK
- J1 pad 12: Net-(J1-Pad12) -> I2C_DATA
- J1 pad 13: Net-(J1-Pad13) -> 3V3
- J1 pad 14: Net-(J1-Pad14) -> GNDD
Routing:
- net Net-(J1-Pad12): track 2.29 -> 0.00 mm
- net I2C_DATA: track 0.00 -> 2.29 mm
- net Net-(J1-Pad14): track 1.74 -> 0.00 mm
- net GNDD: track 0.00 -> 1.74 mm
- net Net-(J1-Pad13): track 1.74 -> 0.00 mm
- net 3V3: track 0.00 -> 1.74 mm
- net Net-(J1-Pad11): track 1.66 -> 0.00 mm
- net I2C_CLOCK: track 0.00 -> 1.66 mm
Other:
- board text added: "CORE64 LED MATRIX (LM) V0.1 2021-02-12 Project information at www.Core64.io Designed by Andy Geppert at www.MachineIdeas.com WS2813 LEDs"
- board text removed: "CORE64 LED MATRIX (LM) V0.5 2021-02-12 Project information at www.Core64.io Designed by Andy Geppert at www.MachineIdeas.com WS2813 LEDs"

Commit message: Finish layout, revise notes
Parts:
- JP1, JP2, XLM3: moved to B.Cu
- moved JP3 78.5 mm to (39.5, 27.4), turned to 180 degrees
- moved JP2 10.4 mm to (-16.8, 40.0), turned to 180 degrees
- moved JP1 9.55 mm to (-9.48, 40.0)
- moved XLM3 9.40 mm to (-29.0, 35.5)
- moved L1 1.40 mm to (-9.48, -36.4)
- moved XLM2 1.17 mm to (-0.69, 40.0)
Connections:
- J1 pad 19: +BATT -> Net-(J1-Pad19)
- J1 pad 20: 5VUSB -> Net-(J1-Pad20)
- J2 pad 19: Net-(J2-Pad19) -> +BATT
- J2 pad 20: Net-(J2-Pad20) -> 5VUSB
Routing:
- net Net-(JP3-Pad1): track 0.00 -> 87.9 mm
- net I2C_CLOCK: track 1.66 -> 89.4 mm, vias 0 -> 1
- net I2C_DATA: track 2.29 -> 84.3 mm, vias 0 -> 2
- net +BATT: track 0.00 -> 78.2 mm
- net 3V3: track 1.74 -> 66.7 mm, vias 0 -> 1
- net GNDD: track 1.74 -> 61.2 mm, vias 0 -> 2
- net Net-(JP2-Pad2): track 0.00 -> 22.5 mm
- net Net-(JP1-Pad2): track 0.00 -> 15.9 mm, vias 0 -> 1
- net 5VUSB: track 0.00 -> 6.37 mm
- net Net-(J1-Pad20): track 0.00 -> 2.00 mm
- net Net-(J1-Pad19): track 0.00 -> 2.00 mm
Other:
- board text added: "+BATT 5VUSB"
- board text added: "1s LiPo Charger"
- board text added: "3V3"
- board text added: "GNDD"
- board text added: "OLED"
- board text added: "SCL SDA"
- board text added: "SCL SDA 3V3 GNDD"
- board text added: "SDA SCL"
- board text added: "SJ1 SJ2"
- board text added: "SJ2 SJ1"

Commit message: Tweak layout and silk screen
Routing:
- net +BATT: track 78.2 -> 85.1 mm
Other:
- outline, holes or cut-outs redrawn
- board text added: "+B"
- board text added: "-B"
- board text added: "5VUSB GND"
- board text added: "ADAFRUIT #1904 MICRO USB ADAFRUIT #4410 USB C"
- board text added: "Battery Limits: 1s or 3.3-7.4V"
- board text added: "CORE64 LED MATRIX (LM) V0.1 2021-02-17 Project information at www.Core64.io Designed by Andy Geppert at www.MachineIdeas.com WS2813 LEDs"
- board text added: "GNDD 3V3 SDA SCL"
- board text added: "J1"
- board text added: "J2"
- board text added: "LSIG USR1"
- board text added: "QWIIC"
- board text added: "USR2 USR3"
- board text added: "XLM2"
- board text added: "XLM4"
- board text removed: "CORE64 LED MATRIX (LM) V0.1 2021-02-12 Project information at www.Core64.io Designed by Andy Geppert at www.MachineIdeas.com WS2813 LEDs"
- board text removed: "LSIG USER"

Commit message: Create BOM and CPL
Parts:
- JP3: value SolderJumper_2_Open -> Teensy_Charge_Enable
- moved L1 1.82 mm to (-11.3, -36.4)
Other:
- board text added: "5VUSB"
- board text added: "Add insulating layer between LiPo Charger and LM PCB."
- board text added: "B+"
- board text added: "B-"
- board text added: "Battery Limits: 1s or 3.3-7.5V"
- board text added: "CORE64 LED MATRIX (LM) V0.1 2021-02-18 Project information at www.Core64.io Designed by Andy Geppert at www.MachineIdeas.com WS2813 LEDs"
- board text added: "LEDS 0-7 ->"
- board text added: "LEDS 56-63 ->"
- board text removed: "0-7 Pixels->"
- board text removed: "63-56 <-bits"
- board text removed: "<-bits 7-0"
- board text removed: "Battery Limits: 1s or 3.3-7.4V"
- board text removed: "CORE64 LED MATRIX (LM) V0.1 2021-02-17 Project information at www.Core64.io Designed by Andy Geppert at www.MachineIdeas.com WS2813 LEDs"
- board text removed: "Pixels-> 56-63"
Changed lines of the file:
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@@
   (general
     (thickness 1.6)
-    (drawings 72)
+    (drawings 75)
     (tracks 1217)
     (zones 0)
@@
     (45 Margin user hide)
     (46 B.CrtYd user hide)
-    (47 F.CrtYd user)
+    (47 F.CrtYd user hide)
     (48 B.Fab user hide)
-    (49 F.Fab user)
+    (49 F.Fab user hide)
   )
   (setup
@@
       (drillshape 0)
       (scaleselection 1)
-      (outputdirectory "Core64_V0.4_Gerbers/"))
+      (outputdirectory "Core64_LM_V0.1_Gerbers/"))
   )
   (net 0 "")
@@
       (effects (font (size 1 1) (thickness 0.15)) (justify mirror))
     )
-    (fp_text value SolderJumper_2_Open (at 0 -1.9) (layer B.Fab)
+    (fp_text value Teensy_Charge_Enable (at 0 -1.9) (layer B.Fab)
       (effects (font (size 1 1) (thickness 0.15)) (justify mirror))
     )
@@
     (tags "Surface mounted pin header SMD 1x16 2.54mm single row style2 pin1 right")
     (attr smd)
-    (fp_text reference J2 (at 0 21.38) (layer B.SilkS)
+    (fp_text reference J2 (at 0 21.02) (layer B.SilkS)
       (effects (font (size 1 1) (thickness 0.15)) (justify mirror))
     )
@@
     (tags "Surface mounted pin header SMD 1x16 2.54mm single row style2 pin1 right")
     (attr smd)
-    (fp_text reference J1 (at 0 21.38) (layer B.SilkS)
+    (fp_text reference J1 (at -2.46 19.02) (layer B.SilkS)
       (effects (font (size 1 1) (thickness 0.15)) (justify mirror))
     )
@@
   )
   (module Core_Memory_8x8_Array:Core64_Logo_9mm_tall (layer F.Cu)
-    (at -9.485 -36.35)
+    (at -11.3 -36.35)
     (fp_text reference L1 (at 0 -12.25) (layer Dwgs.User) hide
       (effects (font (size 1.524 1.524) (thickness 0.3)))
@@
     )
   )
+  (gr_text "Add insulating\nlayer between\nLiPo Charger\nand LM PCB." (at 30.4 -31.6) (layer B.SilkS)
+    (effects (font (size 1.5 1) (thickness 0.16)) (justify left mirror))
+  )
+  (gr_text B+ (at 14.3 -27.9) (layer F.SilkS)
+    (effects (font (size 0.8 0.8) (thickness 0.16)) (justify right))
+  )
+  (gr_text B- (at 14.2 -30.5) (layer F.SilkS)
+    (effects (font (size 0.8 0.8) (thickness 0.16)) (justify right))
+  )
+  (gr_text GND (at 14.2 -33) (layer F.SilkS)
+    (effects (font (size 0.8 0.8) (thickness 0.16)) (justify right))
+  )
+  (gr_text 5VUSB (at 14.3 -35.5) (layer F.SilkS)
+    (effects (font (size 0.8 0.8) (thickness 0.16)) (justify right))
+  )
   (gr_text XLM4 (at -18.925 -30.5) (layer B.SilkS)
     (effects (font (size 1 1) (thickness 0.15)) (justify left mirror))
@@
     (effects (font (size 1.58 0.8) (thickness 0.16)) (justify left mirror))
   )
-  (gr_text J2 (at 35.575 -26.125) (layer F.SilkS)
+  (gr_text J2 (at 33 -24.1) (layer F.SilkS)
     (effects (font (size 1 1) (thickness 0.15)))
   )
-  (gr_text J1 (at -35.5 -26.175) (layer F.SilkS)
+  (gr_text J1 (at -33.1 -24.1) (layer F.SilkS)
     (effects (font (size 1 1) (thickness 0.15)))
   )
@@
     (effects (font (size 1 1) (thickness 0.15)) (justify left mirror))
   )
-  (gr_text "Battery Limits:\n1s or 3.3-7.4V" (at 8.175 -29.325) (layer B.SilkS)
+  (gr_text "Battery Limits:\n1s or 3.3-7.5V" (at 8.175 -29.325) (layer B.SilkS)
     (effects (font (size 1.5 1.5) (thickness 0.3)) (justify left mirror))
   )
@@
   (gr_circle (center 38 -38) (end 39.15 -38) (layer Edge.Cuts) (width 0.05))
   (gr_circle (center -38 38) (end -36.85 38) (layer Edge.Cuts) (width 0.05))
-  (gr_text "0-7\nPixels->" (at -34.485 -28.05) (layer F.SilkS)
+  (gr_text "LEDS 0-7 ->" (at -39.8 -26.7) (layer F.SilkS)
     (effects (font (size 1.6 1) (thickness 0.25)) (justify left))
   )
@@
     (effects (font (size 1.58 0.8) (thickness 0.16)) (justify right))
   )
-  (gr_text www.Core64.io (at -15.975 -39.05) (layer B.SilkS)
+  (gr_text www.Core64.io (at -13 -38.5) (layer B.SilkS)
     (effects (font (size 3.5 3.5) (thickness 0.5)) (justify mirror))
   )
-  (gr_text "63-56\n<-bits" (at 31.715 -27.85) (layer F.SilkS)
-    (effects (font (size 1.6 1) (thickness 0.25)))
-  )
-  (gr_text "<-bits\n   7-0" (at 31.315 28.45) (layer F.SilkS)
-    (effects (font (size 1.6 1) (thickness 0.25)))
-  )
-  (gr_text "Pixels->\n56-63" (at -33.985 28.35) (layer F.SilkS)
+  (gr_text "LEDS 56-63 ->" (at -39.7 27.1) (layer F.SilkS)
     (effects (font (size 1.6 1) (thickness 0.25)) (justify left))
   )
@@
     (arrow2b (pts (xy 42.5 -50.549999) (xy 41.373496 -49.963578)))
   )
-  (gr_text "CORE64 LED MATRIX (LM)     V0.1     2021-02-17\nProject information at www.Core64.io\nDesigned by Andy Geppert at www.MachineIdeas.com\nWS2813 LEDs" (at 0 31.25) (layer B.SilkS)
+  (gr_text "CORE64 LED MATRIX (LM)     V0.1     2021-02-18\nProject information at www.Core64.io\nDesigned by Andy Geppert at www.MachineIdeas.com\nWS2813 LEDs" (at 0 31.25) (layer B.SilkS)
     (effects (font (size 1.2 1.2) (thickness 0.15)) (justify mirror))
   )
