File: Electronic Design/Core64 CB v0.5/Core64 CB v0.5.kicad_pcb (KiCad board)
At the start: 2 copper layers, 85 x 85 mm, 53 parts, among them J1 Digi-Key 77311-420-36LF-ND, J2 Digi-Key 77311-420-36LF-ND, U1 SI7210-B-01, U11 SM353LT, U12 SM353LT, U13 SM353LT, U14 SM353LT, U2 SI7210-B-02, U3 SI7210-B-03, U4 SI7210-B-04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

Commit message: LB Layout refinement for optional hall switches
Parts:
- moved R7 0.08 mm to (-33.2, -39.0)
Routing:
- net 3V3_800mA: track 322.6 -> 319.5 mm
- net GNDD: track 302.9 -> 302.1 mm
Changed lines of the file:
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@@
     (thickness 1.6)
     (drawings 57)
-    (tracks 929)
+    (tracks 928)
     (zones 0)
     (modules 53)
@@
   (layers
     (0 F.Cu signal)
-    (31 B.Cu signal hide)
+    (31 B.Cu signal)
     (32 B.Adhes user hide)
     (33 F.Adhes user hide)
     (34 B.Paste user hide)
     (35 F.Paste user hide)
-    (36 B.SilkS user hide)
+    (36 B.SilkS user)
     (37 F.SilkS user)
-    (38 B.Mask user hide)
-    (39 F.Mask user hide)
+    (38 B.Mask user)
+    (39 F.Mask user)
     (40 Dwgs.User user hide)
     (41 Cmts.User user hide)
@@
     (44 Edge.Cuts user)
     (45 Margin user hide)
-    (46 B.CrtYd user hide)
-    (47 F.CrtYd user hide)
+    (46 B.CrtYd user)
+    (47 F.CrtYd user)
     (48 B.Fab user hide)
     (49 F.Fab user hide)
@@
       (drillshape 0)
       (scaleselection 1)
-      (outputdirectory "Core64_V0.4_Gerbers/"))
+      (outputdirectory "Core64_CB_V0.5_Gerbers/"))
   )
   (net 0 "")
@@
     (tags resistor)
     (attr smd)
-    (fp_text reference R4 (at 2.7 -1.3) (layer B.SilkS)
+    (fp_text reference R4 (at 0 -1.6) (layer B.SilkS)
       (effects (font (size 1 1) (thickness 0.15)) (justify mirror))
     )
@@
     (tags resistor)
     (attr smd)
-    (fp_text reference R3 (at 2.7 -1.3) (layer B.SilkS)
+    (fp_text reference R3 (at 0 -1.5) (layer B.SilkS)
       (effects (font (size 1 1) (thickness 0.15)) (justify mirror))
     )
@@
     (tags resistor)
     (attr smd)
-    (fp_text reference R2 (at 2.7 -1.3) (layer B.SilkS)
+    (fp_text reference R2 (at 0 -1.6) (layer B.SilkS)
       (effects (font (size 1 1) (thickness 0.15)) (justify mirror))
     )
@@
     (tags resistor)
     (attr smd)
-    (fp_text reference R1 (at 2.675 -1.275) (layer B.SilkS)
+    (fp_text reference R1 (at 0 -1.5) (layer B.SilkS)
       (effects (font (size 1 1) (thickness 0.15)) (justify mirror))
     )
@@
     (tags capacitor)
     (attr smd)
-    (fp_text reference C4 (at -2.7 -1.2) (layer B.SilkS)
+    (fp_text reference C4 (at 0 -1.4) (layer B.SilkS)
       (effects (font (size 1 1) (thickness 0.15)) (justify mirror))
     )
@@
     (tags capacitor)
     (attr smd)
-    (fp_text reference C3 (at -2.6 -1.1) (layer B.SilkS)
+    (fp_text reference C3 (at 0 -1.4) (layer B.SilkS)
       (effects (font (size 1 1) (thickness 0.15)) (justify mirror))
     )
@@
     (tags capacitor)
     (attr smd)
-    (fp_text reference C2 (at -2.6 -1.1) (layer B.SilkS)
+    (fp_text reference C2 (at 0 -1.4) (layer B.SilkS)
       (effects (font (size 1 1) (thickness 0.15)) (justify mirror))
     )
@@
     (tags capacitor)
     (attr smd)
-    (fp_text reference C1 (at -2.7 -1.2) (layer B.SilkS)
+    (fp_text reference C1 (at 0 -1.4) (layer B.SilkS)
       (effects (font (size 1 1) (thickness 0.15)) (justify mirror))
     )
@@
   )
   (module Resistor_SMD:R_0805_2012Metric (layer B.Cu)
-    (at -33.21 -38.875 270)
+    (at -33.185 -38.95 270)
     (descr "Resistor SMD 0805 (2012 Metric), square (rectangular) end terminal, IPC_7351 nominal, (Body size source: https://docs.google.com/spreadsheets/d/1BsfQQcO9C6DZCsRaXUlFlo91Tg2WpOkGARC1WS5S8t0/edit?usp=sharing), generated with kicad-footprint-generator")
     (tags resistor)
@@
     (effects (font (size 1 1) (thickness 0.15)) (justify mirror))
   )
-  (gr_text 0x30 (at -22.06 34.1) (layer B.SilkS)
+  (gr_text 0x30 (at -18.185 34.25) (layer B.SilkS)
     (effects (font (size 1 1) (thickness 0.16)) (justify mirror))
   )
-  (gr_text 0x31 (at -8.71 34.225) (layer B.SilkS)
+  (gr_text 0x31 (at -4.685 34.35) (layer B.SilkS)
     (effects (font (size 1 1) (thickness 0.16)) (justify mirror))
   )
-  (gr_text 0x32 (at 4.59 34.225) (layer B.SilkS)
+  (gr_text 0x32 (at 8.715 34.35) (layer B.SilkS)
     (effects (font (size 1 1) (thickness 0.16)) (justify mirror))
   )
-  (gr_text 0x33 (at 18.14 34.25) (layer B.SilkS)
+  (gr_text 0x33 (at 22.115 34.35) (layer B.SilkS)
     (effects (font (size 1 1) (thickness 0.16)) (justify mirror))
   )
@@
   (segment (start -35.56 -6.35) (end -32.585 -6.35) (width 0.6) (layer B.Cu) (net 13))
   (segment (start -29.685 22.6275) (end -28.6875 23.625) (width 0.6) (layer B.Cu) (net 13))
-  (segment (start -30.235 17.1) (end -29.685 17.65) (width 0.6) (layer B.Cu) (net 13))
-  (segment (start -30.235 10.125) (end -30.235 17.1) (width 0.6) (layer B.Cu) (net 13))
+  (segment (start -29.685 17.95) (end -29.685 22.6275) (width 0.6) (layer B.Cu) (net 13))
+  (segment (start -30.235 17.4) (end -29.685 17.95) (width 0.6) (layer B.Cu) (net 13))
+  (segment (start -30.235 10.125) (end -30.235 17.4) (width 0.6) (layer B.Cu) (net 13))
   (segment (start -30.21 10.1) (end -30.235 10.125) (width 0.6) (layer B.Cu) (net 13))
   (segment (start -28.7125 10.1) (end -30.21 10.1) (width 0.6) (layer B.Cu) (net 13))
-  (segment (start -29.685 17.65) (end -29.685 22.6275) (width 0.6) (layer B.Cu) (net 13))
   (segment (start -28.6875 10.125) (end -28.7125 10.1) (width 0.6) (layer B.Cu) (net 13))
   (segment (start -35.56 -8.89) (end -37.215 -8.89) (width 0.6) (layer B.Cu) (net 14))
@@
   (segment (start -2.46 -31.1) (end -2.06 -31.5) (width 0.25) (layer F.Cu) (net 21))
   (segment (start -2.465 -31.1) (end -2.46 -31.1) (width 0.25) (layer F.Cu) (net 21))
-  (segment (start -17.785 -41.85) (end -16.885 -40.95) (width 0.6) (layer B.Cu) (net 21))
-  (segment (start -34.76 -41.85) (end -17.785 -41.85) (width 0.6) (layer B.Cu) (net 21))
-  (segment (start -35.56 -41.05) (end -34.76 -41.85) (width 0.6) (layer B.Cu) (net 21))
-  (segment (start -35.56 -37.525) (end -35.56 -41.05) (width 0.6) (layer B.Cu) (net 21))
-  (segment (start -39.66 -33.425) (end -35.56 -37.525) (width 0.6) (layer B.Cu) (net 21))
-  (segment (start -39.66 -31.5) (end -39.66 -33.425) (width 0.6) (layer B.Cu) (net 21))
   (via (at -35.735 36.625) (size 0.65) (drill 0.35) (layers F.Cu B.Cu) (net 21))
   (segment (start -41.41 30.95) (end -36.059999 36.300001) (width 0.6) (layer F.Cu) (net 21))
@@
   (segment (start 21.964996 -40.465381) (end 21.964996 -40.925) (width 0.3) (layer B.Cu) (net 21))
   (segment (start -19.285 36.65) (end -35.735 36.625) (width 0.6) (layer B.Cu) (net 21))
+  (segment (start -17.785 -41.85) (end -16.885 -40.95) (width 0.6) (layer B.Cu) (net 21))
+  (segment (start -33.385 -41.85) (end -17.785 -41.85) (width 0.6) (layer B.Cu) (net 21))
+  (segment (start -35.56 -39.675) (end -33.385 -41.85) (width 0.6) (layer B.Cu) (net 21))
+  (segment (start -39.66 -33.425) (end -35.56 -37.525) (width 0.6) (layer B.Cu) (net 21))
+  (segment (start -35.56 -37.525) (end -35.56 -39.675) (width 0.6) (layer B.Cu) (net 21))
+  (segment (start -39.66 -31.5) (end -39.66 -33.425) (width 0.6) (layer B.Cu) (net 21))
   (segment (start 30.065 8.7475) (end 28.6875 10.125) (width 0.6) (layer B.Cu) (net 22))
   (segment (start 30.065 -15.4975) (end 30.065 8.7475) (width 0.6) (layer B.Cu) (net 22))
@@
   (segment (start -35.635 -35.399998) (end -34.484999 -36.549999) (width 0.6) (layer B.Cu) (net 26))
   (segment (start -35.635 -34.1) (end -35.635 -35.399998) (width 0.6) (layer B.Cu) (net 26))
-  (segment (start -29.76 -39.45) (end -28.385 -39.45) (width 0.6) (layer B.Cu) (net 26))
-  (segment (start -31.31 -41) (end -29.76 -39.45) (width 0.6) (layer B.Cu) (net 26))
-  (segment (start -34.484999 -40.625001) (end -34.11 -41) (width 0.6) (layer B.Cu) (net 26))
-  (segment (start -34.484999 -36.549999) (end -34.484999 -40.625001) (width 0.6) (layer B.Cu) (net 26))
-  (segment (start -33.21 -40.95) (end -33.26 -41) (width 0.6) (layer B.Cu) (net 26))
-  (segment (start -33.21 -39.9125) (end -33.21 -40.95) (width 0.6) (layer B.Cu) (net 26))
-  (segment (start -33.26 -41) (end -31.31 -41) (width 0.6) (layer B.Cu) (net 26))
-  (segment (start -34.11 -41) (end -33.26 -41) (width 0.6) (layer B.Cu) (net 26))
   (segment (start 3.59 -41.85) (end -27.685 -41.85) (width 0.6) (layer F.Cu) (net 26))
   (via (at 3.59 -41.85) (size 0.65) (drill 0.35) (layers F.Cu B.Cu) (net 26))
@@
   (segment (start -27.460001 33.15) (end -24.37701 33.15) (width 0.6) (layer B.Cu) (net 26))
   (via (at -27.460001 33.15) (size 0.65) (drill 0.35) (layers F.Cu B.Cu) (net 26))
+  (segment (start -30.16 -39.85) (end -29.76 -39.45) (width 0.6) (layer B.Cu) (net 26))
+  (segment (start -33.485 -39.85) (end -30.16 -39.85) (width 0.6) (layer B.Cu) (net 26))
+  (segment (start -29.76 -39.45) (end -28.385 -39.45) (width 0.6) (layer B.Cu) (net 26))
+  (segment (start -34.484999 -38.850001) (end -33.485 -39.85) (width 0.6) (layer B.Cu) (net 26))
+  (segment (start -34.484999 -36.549999) (end -34.484999 -38.850001) (width 0.6) (layer B.Cu) (net 26))
   (segment (start -33.905 3.81) (end -35.56 3.81) (width 0.6) (layer B.Cu) (net 27))
   (segment (start 21.015 37.6) (end 21.015 37.65) (width 0.3) (layer B.Cu) (net 27))
@@
   (via (at -32.51 -35.9) (size 0.65) (drill 0.35) (layers F.Cu B.Cu) (net 64))
   (segment (start -31.66 -35.9) (end -32.51 -35.9) (width 0.3) (layer F.Cu) (net 64))
-  (segment (start -33.235 -36.625) (end -33.235 -38.025) (width 0.3) (layer B.Cu) (net 64))
-  (segment (start -32.51 -35.9) (end -33.235 -36.625) (width 0.3) (layer B.Cu) (net 64))
+  (segment (start -32.86 -38.025) (end -32.885 -38.025) (width 0.3) (layer B.Cu) (net 64))
+  (segment (start -32.885 -38) (end -32.86 -38.025) (width 0.3) (layer B.Cu) (net 64))
+  (segment (start -32.885 -36.275) (end -32.885 -38) (width 0.3) (layer B.Cu) (net 64))
+  (segment (start -32.51 -35.9) (end -32.885 -36.275) (width 0.3) (layer B.Cu) (net 64))
 )

Commit message: Refine and release LB and CB V0.5 layout for prototyping
Parts:
- added U8: LTR-329ALS-01, LiteOn_LTR-329ALS:LTR-329ALS-01, F.Cu at (-35.8, -32.8)
- moved C7 1.88 mm to (-39.6, -32.5)
- renumbered U9 to U10, U8 to U9
Routing:
- net GNDD: track 302.1 -> 306.7 mm, vias 10 -> 11
- net 3V3_800mA: track 319.5 -> 322.4 mm, vias 24 -> 25
- net I2C_DATA: track 222.4 -> 224.1 mm
- net I2C_CLOCK: track 232.8 -> 234.1 mm
Other:
- outline, holes or cut-outs redrawn
- board text added: "CORE BOARD V0.5 2021-02-27 ANDY GEPPERT WWW.MACHINEIDEAS.COM"
- board text added: "HS1/0x30"
- board text added: "HS2/0x31"
- board text added: "HS3/0x32"
- board text added: "HS4/0x33"
- board text removed: "CORE BOARD V0.5 2021-02-15 ANDY GEPPERT WWW.MACHINEIDEAS.COM"
