File: Electronic Design/Core64 LB v0.5/Core64 LB v0.5 Power.sch (KiCad schematic (older format))
At the start: 28 parts, among them IC1 TPS7A0533PDBVR, IC2 LP3961EMP-5.0, IC3 NCP176AMX330TCG, J3 Conn_01x08_Female, J7 S03B-PASK-2_LF__SN_, J8 5V0 Cur. Mon., J9 3V3 Cur. Mon., Q1 MCC_SL3401A, SW1 JS102011SAQN, U6 Micro_LiPo_Charger

Commit message: Connect row-col-0 to analog inputs for self-test mode
Parts:
- removed C14, C3: 1uF, Capacitor_SMD:C_0805_2012Metric, symbol Device:C
- removed IC3: NCP176AMX330TCG, NCP176AMX330TCG:NCP176AMX330TCG, symbol NCP176AMX330TCG:NCP176AMX330TCG
- removed JP8: 3V3_Select, Jumper:SolderJumper-3_P1.3mm_Open_Pad1.0x1.5mm_NumberLabels, symbol Jumper:SolderJumper_3_Open
- added R57, R58: 11k, Resistor_SMD:R_0805_2012Metric, symbol Device:R
Connections:
- net -BATT: now also R58.2
- net 3V3: now also C2.1, IC1.5 (OUT)
- net 5V0: now also R57.1
- new net 5V0_MON: R57.2, R58.1
Other:
- note removed: "Must\nSelect\nOne\nw/SJ"
- note removed: "Preferred, TINY XDFN6\n0.13V DROP @ 500mA"
Changed lines of the file:
@@
 Text Notes 7800 4450 0    118  ~ 0
 3.3V POWER SUPPLY
-$Comp
-L power:GND #PWR0116
-U 1 1 5E8C4F56
-P 9550 6400
-AR Path="/5E7548ED/5E8C4F56" Ref="#PWR0116"  Part="1"
-AR Path="/5E755AC8/5D254AE8/5E8C4F56" Ref="#PWR?"  Part="1"
-F 0 "#PWR0116" H 9550 6150 50  0001 C CNN
-F 1 "GND" H 9555 6225 50  0000 C CNN
-F 2 "" H 9550 6400 50  0001 C CNN
-F 3 "" H 9550 6400 50  0001 C CNN
-	1    9550 6400
-	-1   0    0    -1
-$EndComp
 Wire Notes Line
 	5200 850  5200 3750
@@
 Wire Wire Line
 	3850 5850 3850 5900
-$Comp
-L Device:C C?
-U 1 1 5EBB7068
-P 7750 6150
-AR Path="/5E755787/5EBB7068" Ref="C?"  Part="1"
-AR Path="/5E755AC8/5D2551FF/5EBB7068" Ref="C?"  Part="1"
-AR Path="/5EA63449/5EBB7068" Ref="C?"  Part="1"
-AR Path="/5E7548ED/5EBB7068" Ref="C3"  Part="1"
-F 0 "C3" H 7841 6196 50  0000 L CNN
-F 1 "1uF" H 7841 6105 50  0000 L CNN
-F 2 "Capacitor_SMD:C_0805_2012Metric" H 7750 6150 50  0001 C CNN
-F 3 "~" H 7750 6150 50  0001 C CNN
-	1    7750 6150
-	-1   0    0    -1
-$EndComp
 $Comp
 L Device:C C?
@@
 All non-polarized capacitors are X7R or X5R ceramic unless otherwise noted.
 $Comp
-L NCP176AMX330TCG:NCP176AMX330TCG IC3
-U 1 1 5F5A7E01
-P 9250 6000
-F 0 "IC3" H 9850 6268 50  0000 C CNN
-F 1 "NCP176AMX330TCG" H 9850 6175 50  0000 C CNN
-F 2 "NCP176AMX330TCG:NCP176AMX330TCG" H 10300 6100 50  0001 L CNN
-F 3 "https://www.mouser.com/datasheet/2/308/NCP176-D-1551588.pdf" H 10300 6000 50  0001 L CNN
-F 4 "ON Semiconductor NCP176AMX330TCG, LDO Voltage Regulator, 500mA, 3.3 V +/-0.8%, 1.4  5.5 Vin, 6-Pin XDFN" H 10300 5900 50  0001 L CNN "Description"
-F 5 "0.45" H 10300 5800 50  0001 L CNN "Height"
-F 6 "ON Semiconductor" H 10300 5700 50  0001 L CNN "Manufacturer_Name"
-F 7 "NCP176AMX330TCG" H 10300 5600 50  0001 L CNN "Manufacturer_Part_Number"
-F 8 "NCP176AMX330TCG" H 10300 5500 50  0001 L CNN "Arrow Part Number"
-F 9 "https://www.arrow.com/en/products/ncp176amx330tcg/on-semiconductor" H 10300 5400 50  0001 L CNN "Arrow Price/Stock"
-F 10 "863-NCP176AMX330TCG" H 10300 5300 50  0001 L CNN "Mouser Part Number"
-F 11 "https://www.mouser.com/Search/Refine.aspx?Keyword=863-NCP176AMX330TCG" H 10300 5200 50  0001 L CNN "Mouser Price/Stock"
-	1    9250 6000
-	-1   0    0    -1
-$EndComp
-$Comp
 L TPS7A0533PDBVR:TPS7A0533PDBVR IC1
 U 1 1 5F5B23D2
@@
 	1    0    0    -1
 $EndComp
-Text Notes 8250 5700 0    50   ~ 0
-Preferred, TINY XDFN6\n0.13V DROP @ 500mA
 Text Notes 8250 4750 0    50   ~ 0
 Alternate, SOT-23-5\n0.24V DROP @ 200mA
@@
 F 3 "" H 7850 5300 50  0001 C CNN
 	1    7850 5300
-	1    0    0    -1
-$EndComp
-Wire Wire Line
-	9250 6100 9300 6100
-Wire Wire Line
-	9300 6100 9300 6000
-Wire Wire Line
-	9300 6000 9250 6000
-Connection ~ 9300 6000
-$Comp
-L Device:C C?
-U 1 1 5F5D4D85
-P 9550 6200
-AR Path="/5E755787/5F5D4D85" Ref="C?"  Part="1"
-AR Path="/5E755AC8/5D2551FF/5F5D4D85" Ref="C?"  Part="1"
-AR Path="/5EA63449/5F5D4D85" Ref="C?"  Part="1"
-AR Path="/5E7548ED/5F5D4D85" Ref="C14"  Part="1"
-F 0 "C14" H 9641 6246 50  0000 L CNN
-F 1 "1uF" H 9641 6155 50  0000 L CNN
-F 2 "Capacitor_SMD:C_0805_2012Metric" H 9550 6200 50  0001 C CNN
-F 3 "~" H 9550 6200 50  0001 C CNN
-	1    9550 6200
 	1    0    0    -1
 $EndComp
@@
 $EndComp
 Wire Wire Line
-	9250 6300 9400 6300
-Wire Wire Line
-	9400 6300 9400 5850
-Wire Wire Line
-	9300 6000 9550 6000
-Text GLabel 9400 5850 1    50   Input ~ 0
-5V0
-Wire Wire Line
-	9550 6000 9550 6050
-Connection ~ 9550 6000
-Wire Wire Line
-	9550 6350 9550 6400
-$Comp
-L power:GND #PWR0125
-U 1 1 5F5EF2E5
-P 7900 6400
-AR Path="/5E7548ED/5F5EF2E5" Ref="#PWR0125"  Part="1"
-AR Path="/5E755AC8/5D254AE8/5F5EF2E5" Ref="#PWR?"  Part="1"
-F 0 "#PWR0125" H 7900 6150 50  0001 C CNN
-F 1 "GND" H 7905 6225 50  0000 C CNN
-F 2 "" H 7900 6400 50  0001 C CNN
-F 3 "" H 7900 6400 50  0001 C CNN
-	1    7900 6400
-	-1   0    0    -1
-$EndComp
-Wire Wire Line
-	8050 6100 7900 6100
-Wire Wire Line
-	8050 6200 7900 6200
-Wire Wire Line
-	7900 6200 7900 6350
-Wire Wire Line
-	7750 6000 7750 5950
-Wire Wire Line
-	7750 5950 7900 5950
-Connection ~ 7900 5950
-Wire Wire Line
-	7750 6300 7750 6350
-Wire Wire Line
-	7750 6350 7900 6350
-Connection ~ 7900 6350
-Wire Wire Line
-	7900 6350 7900 6400
-Wire Wire Line
 	9150 5150 9250 5150
 $Comp
@@
 Wire Wire Line
 	7850 5250 7850 5300
-$Comp
-L Jumper:SolderJumper_3_Open JP8
-U 1 1 5F67458E
-P 9700 5550
-F 0 "JP8" V 9600 5650 50  0000 L CNN
-F 1 "3V3_Select" V 9950 5100 50  0000 L CNN
-F 2 "Jumper:SolderJumper-3_P1.3mm_Open_Pad1.0x1.5mm_NumberLabels" H 9700 5550 50  0001 C CNN
-F 3 "~" H 9700 5550 50  0001 C CNN
-	1    9700 5550
-	0    -1   -1   0
-$EndComp
-Wire Wire Line
-	9700 5350 9700 4800
 Wire Wire Line
 	9400 4800 9700 4800
-Wire Wire Line
-	9700 6000 9700 5750
-Wire Wire Line
-	9550 6000 9700 6000
-Text Notes 9800 5200 0    118  ~ 24
-Must\nSelect\nOne\nw/SJ
 Text GLabel 8000 4650 0    50   Input ~ 0
-5V0
-Text GLabel 7850 5750 0    50   Input ~ 0
 5V0
 $Comp
@@
 Connection ~ 7100 5500
 Wire Wire Line
-	7850 5750 7900 5750
-Wire Wire Line
-	7900 5750 7900 5950
-Wire Wire Line
 	8000 4650 8100 4650
 Wire Wire Line
 	8100 4650 8100 4800
-Wire Wire Line
-	7900 5950 7900 6100
 Wire Wire Line
 	7100 5500 7100 5750
@@
 	0    -1   1    0
 $EndComp
-Wire Wire Line
-	9250 6200 9300 6200
-Wire Wire Line
-	9300 6200 9300 6450
-Wire Wire Line
-	9300 6450 8050 6450
-Wire Wire Line
-	8050 6450 8050 6350
-Wire Wire Line
-	8050 6350 7900 6350
 Connection ~ 7100 5000
 Wire Wire Line
@@
 Wire Wire Line
 	650  3150 5100 3150
-Wire Wire Line
-	5100 3150 5100 2600
 Wire Wire Line
 	5100 2600 6650 2600
@@
 Text Notes 5700 6200 0    50   ~ 0
 0.24V DROP @ 800mA
-Text Notes 7650 5650 0    50   ~ 0
+Text Notes 7550 4550 0    50   ~ 0
 IN MAX 5.5V
 Wire Wire Line
@@
 Wire Wire Line
 	4050 4100 4900 4100
-Wire Wire Line
-	9850 5550 10000 5550
 Wire Wire Line
 	10100 5550 10200 5550
@@
 Text GLabel 1500 4100 2    50   Input ~ 0
 TEENSY_VUSB
+$Comp
+L Device:R R?
+U 1 1 603A6799
+P 7550 5850
+AR Path="/5E755787/603A6799" Ref="R?"  Part="1"
+AR Path="/5E755AC8/5D2551FF/603A6799" Ref="R?"  Part="1"
+AR Path="/5E7548ED/603A6799" Ref="R57"  Part="1"
+F 0 "R57" H 7620 5896 50  0000 L CNN
+F 1 "11k" H 7620 5805 50  0000 L CNN
+F 2 "Resistor_SMD:R_0805_2012Metric" V 7480 5850 50  0001 C CNN
+F 3 "~" H 7550 5850 50  0001 C CNN
+	1    7550 5850
+	1    0    0    -1
+$EndComp
+$Comp
+L Device:R R?
+U 1 1 603A679F
+P 7550 6150
+AR Path="/5E755787/603A679F" Ref="R?"  Part="1"
+AR Path="/5E755AC8/5D2551FF/603A679F" Ref="R?"  Part="1"
+AR Path="/5E7548ED/603A679F" Ref="R58"  Part="1"
+F 0 "R58" H 7620 6196 50  0000 L CNN
+F 1 "11k" H 7620 6105 50  0000 L CNN
+F 2 "Resistor_SMD:R_0805_2012Metric" V 7480 6150 50  0001 C CNN
+F 3 "~" H 7550 6150 50  0001 C CNN
+	1    7550 6150
+	1    0    0    -1
+$EndComp
+Wire Wire Line
+	7800 6000 7550 6000
+Text GLabel 7800 6000 2    50   Output ~ 0
+5V0_MON
+$Comp
+L power:GND #PWR0159
+U 1 1 603A67A7
+P 7550 6350
+AR Path="/5E7548ED/603A67A7" Ref="#PWR0159"  Part="1"
+AR Path="/5E755AC8/5D254AE8/603A67A7" Ref="#PWR?"  Part="1"
+F 0 "#PWR0159" H 7550 6100 50  0001 C CNN
+F 1 "GND" H 7555 6175 50  0000 C CNN
+F 2 "" H 7550 6350 50  0001 C CNN
+F 3 "" H 7550 6350 50  0001 C CNN
+	1    7550 6350
+	1    0    0    -1
+$EndComp
+Wire Wire Line
+	7550 6300 7550 6350
+Connection ~ 7550 6000
+Text Notes 7850 6200 0    50   ~ 0
+1%
+Text Notes 7850 5900 0    50   ~ 0
+1%
+Text GLabel 7500 5600 0    50   Output ~ 0
+5V0
+Wire Wire Line
+	7500 5600 7550 5600
+Wire Wire Line
+	7550 5600 7550 5700
+Wire Wire Line
+	9000 6000 8750 6000
+Text GLabel 9000 6000 2    50   Output ~ 0
+3V3_MON
+Text GLabel 8750 6000 0    50   Output ~ 0
+3V3
+Wire Wire Line
+	9700 4800 9700 5550
+Wire Wire Line
+	9700 5550 10000 5550
+Wire Wire Line
+	5100 3150 5100 2600
 $EndSCHEMATC

Commit message: LB layout redlines
Parts:
- SW1: footprint Button_Switch_SMD:SW_SPDT_CK-JS102011SAQN -> Button_Switch_SMD:SW_SPDT_CK-JS102011SAQN_Core64_Recessed
Connections:
- net VBAT_MON renamed BAT_MON
Changed lines of the file:
@@
 F 0 "SW1" H 1500 5550 50  0000 C CNN
 F 1 "JS102011SAQN" H 1500 5450 50  0000 C CNN
-F 2 "Button_Switch_SMD:SW_SPDT_CK-JS102011SAQN" H 1450 5250 50  0001 C CNN
+F 2 "Button_Switch_SMD:SW_SPDT_CK-JS102011SAQN_Core64_Recessed" H 1450 5250 50  0001 C CNN
 F 3 "~" H 1450 5250 50  0001 C CNN
 	1    1450 5250
@@
 	4100 5550 3850 5550
 Text GLabel 4100 5550 2    50   Output ~ 0
-VBAT_MON
+BAT_MON
 Text Notes 650  6850 0    118  ~ 0
 ALL SYSTEM GROUND
@@
 *** ALL CONFIGURATIONS REQUIRE\nCUTTING VIN-VUSB TRACE ON\nBACK OF TEENSY ***
 Text GLabel 5400 7450 1    50   Output ~ 0
-VBAT_MON
+BAT_MON
 Text Notes 7600 3150 0    157  ~ 31
 1S LIPO ONLY !!!

Commit message: Move LiPo Charger to top edge, increase LCD footprint top header edge up 1mm
Parts:
- U6: footprint Core_Memory_8x8_Array:Micro_LiPo_Charger -> Core_Memory_8x8_Array:Micro_LiPo_Charger_CornerSMD
Changed lines of the file:
@@
 F 0 "U6" V 5650 3200 50  0000 L CNN
 F 1 "Micro_LiPo_Charger" V 5500 2650 50  0000 L CNN
-F 2 "Core_Memory_8x8_Array:Micro_LiPo_Charger" H 5800 3000 50  0001 C CNN
+F 2 "Core_Memory_8x8_Array:Micro_LiPo_Charger_CornerSMD" H 5800 3000 50  0001 C CNN
 F 3 "" H 5800 3000 50  0001 C CNN
 	1    5800 3000

Commit message: Update schematic battery and LiPo charger notes, move SD_CD from ANA_6 to SPARE_3, schematic red lines
Parts:
- J7: footprint JST_S03B-PASK-2_LF__SN_:S03BPASK2LFSN -> JST_S03B-PASK-2_LF__SN_:S03BPASK2LFSN_.075in_holes
- JP5: footprint Jumper:SolderJumper-2_P1.3mm_Bridged_RoundedPad1.0x1.5mm -> Jumper:SolderJumper-2_P1.3mm_Open_RoundedPad1.0x1.5mm; symbol Jumper:SolderJumper_2_Bridged -> Jumper:SolderJumper_2_Open
- Q1: symbol Device:Q_PMOS_DGS -> Device:Q_PMOS_GSD
Connections:
- net +RPP: now also Q1.2 (S); no longer Q1.3 (S)
- net at C8.1, SW1.2 (B): now also Q1.3 (D); no longer Q1.1 (D)
- net at R48.1, Z1.2 (A): now also Q1.1 (G); no longer Q1.2 (G)
Other:
- note added: "1) Remove the 4x “AAA” battery pack AND the battery connector.\n2) Purchase and install a LiPo charge manager.\n a) The board is designed to accept this one: https://www.adafruit.com/product/1904 (Micro USB) and 4410 (USB C).\n b) Solder the the charge manager directly to the board to keep a low profile.\n3) Purchase and install a 1S LiPo using double-sided tape. \n a) Choose a 1S Lipo with built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"
- note added: "1S LIPO ONLY !!!\nDo NOT connect AAAs to a LiPo charger!\nYou will destroy the charging chip."
- note added: "OPT: Close SJ to run board\nwhile it is charging with the\nLiPo charger USB port."
- note added: "SOT-23-5\n0.24V DROP @ 200mA"
- note added: "SOURCE 1 “ON (BAT)”\n BUILT-IN BATTERY PACK (Keystone 2482CN) WITH 4X “AAA” Primary/Alkaline Cells\n OK to use Energizer Ultimate Lithium (light weight!) with open cell 7.2V, loaded will be <7V.\n Battery Pack includes wires and may or may not have a 3-pin plug.\n \n Optional Socket: TH, Side Entry, JST PA S03B-PASK-2(LF)(SN), Digikey 455-1848-ND\n"
- note added: "SOURCE 2 “OFF (USB)”\n USB 5V supplied through Teensy and optional LiPo Charger USB port.\n With the VIN-VUSB trace cut on the back of the Teensy, the TEENSY_VUSB is taken off of the\n Teensy Board and routed on the Core64 LB to the lower position of the power switch. From\n here, it powers the whole Core64 system and routes back to the TEENSY_VIN after passing\n through the 5V LDO regulator."
- note removed: "1) Remove the 4x “AAA” battery pack AND the battery connector (so you don’t try to charge AAAs with a LiPo charger!).\n\n2) Purchase and install a LiPo charge manager.\n a) The logic board is designed to accept this one: https://www.adafruit.com/product/1904.\n b) Solder the the charge manager directly to the board without headers to keep a low profile to allow the stylus to fit.\n\n3) Purchase a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"
- note removed: "1S LIPO ONLY !!!"
- note removed: "All non-polarized capacitors are X7R or X5R ceramic unless otherwise noted."
- note removed: "Alternate, SOT-23-5\n0.24V DROP @ 200mA"
- note removed: "OPT: Open SJ to disable charging\nfrom TEENSY_VUSB. The USB port\non the charge manager will still work."
- note removed: "SOURCE 1 “ON (BAT)”\n BUILT-IN BATTERY PACK (Keystone 2482CN) WITH 4X “AAA” Primary/Alkaline Cells\n OK to use Energizer Ultimate Lithium (light weight!) with open cell 7.2V, loaded will be <7V.\n Battery Pack includes wires and 3-pin plug.\n \n Socket: TH, Side Entry, JST PA S03B-PASK-2(LF)(SN), Digikey 455-1848-ND ($0.44/ea)\n Socket: SMT, Top Entry, JST PA BM03B-PASS-1-TFT(LF)(SN), Digikey 455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"
- note removed: "SOURCE 2 “OFF (USB)”\n USB 5V supplied through Teensy 3.2 and optional LiPo Charger USB port.\n With the VIN-VUSB trace cut on the back of the Teensy, the TEENSY_VUSB is taken off of the\n Teensy Board and routed on the Core64 LB to the lower position of the power switch. From\n here, it powers the whole Core64 system and routes back to the TEENSY_VIN after passing\n through the 5V LDO regulator."
- moved on the sheet: R57, R58, U6

Commit message: Refine and release LB and CB V0.5 layout for prototyping
Parts:
- JP7: footprint Jumper:SolderJumper-2_P1.3mm_Bridged_Pad1.0x1.5mm -> Jumper:SolderJumper-2_P1.3mm_Bridged_RoundedPad1.0x1.5mm
Other:
- note added: "SOURCE 1 “ON (BAT)”\n BUILT-IN BATTERY PACK (Keystone 2482 or 2482CN) WITH 4X “AAA” primary/Alkaline Cells\n OK to use Energizer Ultimate Lithium (light weight!) with open cell 7.2V, loaded will be <7V.\n Battery Pack includes wires and may or may not have a 3-pin plug.\n \n Optional Socket: TH, Side Entry, JST PA S03B-PASK-2(LF)(SN), Digikey 455-1848-ND\n"
- note removed: "SOURCE 1 “ON (BAT)”\n BUILT-IN BATTERY PACK (Keystone 2482CN) WITH 4X “AAA” Primary/Alkaline Cells\n OK to use Energizer Ultimate Lithium (light weight!) with open cell 7.2V, loaded will be <7V.\n Battery Pack includes wires and may or may not have a 3-pin plug.\n \n Optional Socket: TH, Side Entry, JST PA S03B-PASK-2(LF)(SN), Digikey 455-1848-ND\n"
Changed lines of the file:
@@
 Sheet 4 5
 Title "Core 64 - Power Schematic"
-Date "2021-02-26"
+Date "2021-02-27"
 Rev "0.5"
 Comp "Concept and design by Andy Geppert @ www.MachineIdeas.com"
 Comment1 "Visit www.Core64.io for information on assembly and optional features."
-Comment2 "*** Work in progress ***"
+Comment2 "*** As prototyped. ***"
 Comment3 ""
 Comment4 "All non-polarized capacitors are X7R or X5R ceramic unless otherwise noted."
@@
 $EndComp
 Text Notes 750  1550 0    50   ~ 0
-SOURCE 1 “ON (BAT)”\n  BUILT-IN BATTERY PACK (Keystone 2482CN) WITH 4X “AAA” Primary/Alkaline Cells\n  OK to use Energizer Ultimate Lithium (light weight!) with open cell 7.2V, loaded will be <7V.\n  Battery Pack includes wires and may or may not have a 3-pin plug.\n    \n  Optional Socket: TH, Side Entry, JST PA S03B-PASK-2(LF)(SN), Digikey 455-1848-ND\n
+SOURCE 1 “ON (BAT)”\n  BUILT-IN BATTERY PACK (Keystone 2482 or 2482CN) WITH 4X “AAA” primary/Alkaline Cells\n  OK to use Energizer Ultimate Lithium (light weight!) with open cell 7.2V, loaded will be <7V.\n  Battery Pack includes wires and may or may not have a 3-pin plug.\n    \n  Optional Socket: TH, Side Entry, JST PA S03B-PASK-2(LF)(SN), Digikey 455-1848-ND\n
 Text Notes 750  2950 0    50   ~ 0
 SOURCE 2 “OFF (USB)”\n  USB 5V supplied through Teensy and optional LiPo Charger USB port.\n  With the VIN-VUSB trace cut on the back of the Teensy, the TEENSY_VUSB is taken off of the\n  Teensy Board and routed on the Core64 LB to the lower position of the power switch. From\n  here, it powers the whole Core64 system and routes back to the TEENSY_VIN after passing\n  through the 5V LDO regulator.
@@
 F 0 "JP7" H 950 5500 50  0000 C CNN
 F 1 "USB_Power_Enable" H 850 5600 50  0000 C CNN
-F 2 "Jumper:SolderJumper-2_P1.3mm_Bridged_Pad1.0x1.5mm" H 950 5350 50  0001 C CNN
+F 2 "Jumper:SolderJumper-2_P1.3mm_Bridged_RoundedPad1.0x1.5mm" H 950 5350 50  0001 C CNN
 F 3 "~" H 950 5350 50  0001 C CNN
 	1    950  5350
