File: Electronic Design/Core64 LB v0.5/Core64 LB v0.5 Sense_LEDs_ID.sch (KiCad schematic (older format))
At the start: 25 parts, among them J1 HEADER_8-PIN_0.1, J10 TSM-106-03-T-DV‎, J17 LED Cur. Mon., U1 74HC02, U3 LM393, U3 SN74LV1T125DBVR, U4 M24C01-RMN, U7 LM393

Commit message: Update schematic battery and LiPo charger notes, move SD_CD from ANA_6 to SPARE_3, schematic red lines
Connections:
- net LED_ARRAY_3V3_SIG renamed LED_MATRIX_3V3_SIG
- net LED_ARRAY_5V0_SIG renamed LED_MATRIX_5V0_SIG
Other:
- note added: "LED MATRIX DRIVE AND LEVEL SHIFT"
- note added: "SILKSCREEN: \n5V0 ONLY\nLED MATRIX"
- note removed: "LED ARRAY DRIVE AND LEVEL SHIFT"
- note removed: "SILKSCREEN: \n5V0 ONLY\nLED ARRAY"
Changed lines of the file:
@@
 Date "2021-02-04"
 Rev "0.5"
-Comp "www.Core64.io"
-Comment1 "Work in progress"
-Comment2 "Andy Geppert"
+Comp "Concept and design by Andy Geppert @ www.MachineIdeas.com"
+Comment1 "Visit www.Core64.io for information on assembly and optional features."
+Comment2 "*** Work in progress ***"
 Comment3 ""
-Comment4 ""
+Comment4 "All non-polarized capacitors are X7R or X5R ceramic unless otherwise noted."
 $EndDescr
 Text Notes 600  850  0    118  ~ 0
@@
 NOR -> NOT -> RS LATCH
 Text GLabel 2400 5500 2    50   Output ~ 0
-LED_ARRAY_5V0_SIG
+LED_MATRIX_5V0_SIG
 Wire Wire Line
 	2300 5500 2400 5500
 Text GLabel 1400 5500 0    50   Input ~ 0
-LED_ARRAY_3V3_SIG
+LED_MATRIX_3V3_SIG
 Wire Wire Line
 	1450 6000 1500 6000
@@
 Connection ~ 1900 6350
 Text Notes 600  5250 0    118  ~ 0
-LED ARRAY DRIVE AND LEVEL SHIFT
+LED MATRIX DRIVE AND LEVEL SHIFT
 Wire Wire Line
 	2300 6000 2300 5950
@@
 TSM-106 (2x6) required\nTSM-107 (2x7) alternate\n\nSymbol view is looking down\non the front face of the Logic\nBoard, with the male header\npins pointing up at you.
 Text Notes 2500 6200 0    50   ~ 0
-SILKSCREEN: \n5V0 ONLY\nLED ARRAY
+SILKSCREEN: \n5V0 ONLY\nLED MATRIX
 Wire Wire Line
 	4650 5650 4650 5750
@@
 $EndComp
 Text GLabel 4300 6250 2    50   Input ~ 0
-LED_ARRAY_5V0_SIG
+LED_MATRIX_5V0_SIG
 $Comp
 L Connector_Generic:Conn_02x07_Odd_Even J?

Commit message: Refine and release LB and CB V0.5 layout for prototyping
Other:
- note removed: "All non-polarized capacitors are X7R or X5R ceramic unless otherwise noted."
Changed lines of the file:
@@
 Sheet 2 5
 Title "Core 64 - Sense"
-Date "2021-02-04"
+Date "2021-02-27"
 Rev "0.5"
 Comp "Concept and design by Andy Geppert @ www.MachineIdeas.com"
 Comment1 "Visit www.Core64.io for information on assembly and optional features."
-Comment2 "*** Work in progress ***"
+Comment2 "*** As prototyped. ***"
 Comment3 ""
 Comment4 "All non-polarized capacitors are X7R or X5R ceramic unless otherwise noted."
@@
 	3900 1450 3650 1450
 Connection ~ 3650 1450
-Text Notes 6300 6750 0    50   ~ 0
-All non-polarized capacitors are X7R or X5R ceramic unless otherwise noted.
 Text Notes 8650 2950 0    50   ~ 0
 SILKSCREEN: 3V3 ONLY\nSENSE DEBUG

Commit message: Update schematic and BOM hardware ID EEPROM from 128 to 256 Byte
Parts:
- U4: value M24C01-RMN -> M24C02-RMN
Changed lines of the file:
@@
 AR Path="/5E75D6AB/5F823906" Ref="U4"  Part="1"
 F 0 "U4" H 8800 6300 50  0000 C CNN
-F 1 "M24C01-RMN" H 9450 6300 50  0000 C CNN
+F 1 "M24C02-RMN" H 9450 6300 50  0000 C CNN
 F 2 "Package_SO:SOIC-8_3.9x4.9mm_P1.27mm" H 9100 6350 50  0001 C CNN
 F 3 "http://www.st.com/content/ccc/resource/technical/document/datasheet/b0/d8/50/40/5a/85/49/6f/DM00071904.pdf/files/DM00071904.pdf/jcr:content/translations/en.DM00071904.pdf" H 9150 5500 50  0001 C CNN
