File: Electronic Design/Core64 LM v0.2/Core64 LM v0.2.sch (KiCad schematic (older format))
At the start: 75 parts, among them J1 PASS THROUGH BOARD, J2 PASS THROUGH BOARD

Commit message: Release LM V0.2 Gerbers and assembly files
Changed lines of the file:
@@
 Sheet 1 2
 Title "Core64 LM (LED MATRIX)"
-Date "2021-03-08"
+Date "2021-03-21"
 Rev "0.2"
 Comp "Concept and design by Andy Geppert @ www.MachineIdeas.com"
 Comment1 "Visit www.Core64.io for information on assembly and optional features."
-Comment2 "*** As released 2021-03-xx ***"
+Comment2 "*** As released 2021-03-21 ***"
 Comment3 ""
 Comment4 "All capacitors ceramic X7R unless otherwise noted."
@@
 Wire Wire Line
 	1850 7600 2050 7600
+Connection ~ 9350 700
+Connection ~ 9350 2200
+Connection ~ 9350 2950
+Connection ~ 9350 3700
+Connection ~ 9350 4450
+Connection ~ 9350 5200
+Connection ~ 9350 5950
 $EndSCHEMATC
