File: Electronic Design/Core64 LM v0.3/Core64 LM v0.3.sch (KiCad schematic (older format))
At the start: 75 parts, among them J1 MOST CONNECTIONS PASS THROUGH, J2 MOST CONNECTIONS PASS THROUGH

Commit message: Add opt. 5V0 buffer cap SMD and T.H., add PCB P/N, move corner holes to 37.7mm, move diffuser alignment mount points out and disconnect from GND, silkscreen cleanup
Parts:
- J1, J2: value MOST CONNECTIONS PASS THROUGH -> TSW-108-15-T-S; Manufacturer (none) -> Samtec Inc.; Mfr P/N (none) -> TSW-108-15-T-S
Other:
- note added: "Male headers 1x8 pins,\ncut into 4 pairs and\ninstall at four corners."
Changed lines of the file:
@@
 Sheet 1 2
 Title "Core64 LM (LED MATRIX)"
-Date "2021-05-17"
+Date "2021-08-07"
 Rev "0.3"
 Comp "Concept and design by Andy Geppert @ www.MachineIdeas.com"
@@
 P 1450 6900
 F 0 "J2" V 1400 7700 50  0000 C CNN
-F 1 "MOST CONNECTIONS PASS THROUGH" V 1400 6600 50  0000 C CNN
+F 1 "TSW-108-15-T-S" V 1400 6600 50  0000 C CNN
 F 2 "Connector_PinHeader_2.54mm:PinHeader_1x20_P2.54mm_Vertical_SMD_and_TH_Pin1Right" H 1450 6900 50  0001 C CNN
 F 3 "~" H 1450 6900 50  0001 C CNN
+F 4 "Samtec Inc." H 1450 6900 50  0001 C CNN "Manufacturer"
+F 5 "TSW-108-15-T-S" H 1450 6900 50  0001 C CNN "Mfr P/N"
 	1    1450 6900
 	0    -1   1    0
@@
 P 1450 7900
 F 0 "J1" V 1400 8700 50  0000 C CNN
-F 1 "MOST CONNECTIONS PASS THROUGH" V 1400 7600 50  0000 C CNN
+F 1 "TSW-108-15-T-S" V 1400 7600 50  0000 C CNN
 F 2 "Connector_PinHeader_2.54mm:PinHeader_1x20_P2.54mm_Vertical_SMD_and_TH_Pin1Right" H 1450 7900 50  0001 C CNN
 F 3 "~" H 1450 7900 50  0001 C CNN
+F 4 "Samtec Inc." H 1450 7900 50  0001 C CNN "Manufacturer"
+F 5 "TSW-108-15-T-S" H 1450 7900 50  0001 C CNN "Mfr P/N"
 	1    1450 7900
 	0    -1   -1   0
@@
 Connection ~ 9350 5200
 Connection ~ 9350 5950
+Text Notes 2550 7950 0    50   ~ 0
+Male headers 1x8 pins,\ncut into 4 pairs and\ninstall at four corners.
 $EndSCHEMATC

Commit message: Core64 LED Matrix V0.3 release to manufacturing
Parts:
- C1, C2, C3, C4, C5, C6, C7, C8: INSERT? (none) -> YES; JLCPCB P/N (none) -> C14663; Manufacturer (none) -> YAGEO; Mfr P/N (none) -> CC0603KRX7R9BB104
- D1, D10, D11, D12, D13, D14, D15, D16, D17, D18, D19, D2, D20, D21, D22, D23, D24, D25, D26, D27, D28, D29, D3, D30, D31, D32, D33, D34, D35, D36, D37, D38, D39, D4, D40, D41, D42, D43, D44, D45, D46, D47, D48, D49, D5, D50, D51, D52, D53, D54, D55, D56, D57, D58, D59, D6, D60, D61, D62, D63, D64, D7, D8, D9: value WS2813 -> WS2813C; INSERT? (none) -> YES; JLCPCB P/N (none) -> C194323
- J1, J2, L1: INSERT? (none) -> NO
Other:
- note added: "CORE64 LED MATRIX (LM)\nProject information at www.Core64.io\nDesigned by Andy Geppert | www.MachineIdeas.com\nPCB P/N: 132-001 \nVersion (Date)\nLEDS: WS2813C"
- note added: "SILKSCREEN:\nLEDS/PIXEL 0-7..\nORDER -> 56-63"
- note removed: "CORE64 LED MATRIX (LM)\nProject information at www.Core64.io\nDesigned by Andy Geppert at www.MachineIdeas.com\nPCB P/N: 132-001 \nVersion (Date)\nWS2813 LEDs"
- note removed: "SILKSCREEN:\nLEDS 0-7\nLEDS 8-15…\nLEDS 56-63"
