File: Electronic Design/Core64 CB v0.6/Core64 CB v0.6 Optional.sch (KiCad schematic (older format))
At the start: 34 parts, among them U10 TS3A4751PWR, U11 SM353LT, U12 SM353LT, U13 SM353LT, U14 LTR-329ALS-01, U6 BH1730FVC, U7 LTR-303ALS-01, U8 SM353LT, U9 TS3A4751PWR, X1 SFH11-NBPC-D03-ST-BK

Commit message: CB refine silkscreen, change center ALS BH1730 opening to drill hole and remove center solder pad, clean-up ref. des. numbers
Parts:
- renumbered C7 to C6, C8 to C7, C9 to C8, R7 to R5, U11 to U10, U12 to U11, U13 to U12, U9 to U13, U10 to U14, U14 to U8, U8 to U9
Changed lines of the file:
@@
 Sheet 2 2
 Title "Core64 CB (Core Board)"
-Date "2021-06-07"
+Date "2021-08-08"
 Rev "0.6"
 Comp "Concept and design by Andy Geppert @ www.MachineIdeas.com"
@@
 P 9500 4900
 AR Path="/604F7C67" Ref="C?"  Part="1"
-AR Path="/604D6360/604F7C67" Ref="C7"  Part="1"
-F 0 "C7" H 9250 4950 50  0000 L CNN
+AR Path="/604D6360/604F7C67" Ref="C6"  Part="1"
+F 0 "C6" H 9250 4950 50  0000 L CNN
 F 1 "0.1uF" H 9150 4850 50  0000 L CNN
 F 2 "Capacitor_SMD:C_0805_2012Metric" H 9538 4750 50  0001 C CNN
@@
 P 10900 4900
 AR Path="/604F7C86" Ref="R?"  Part="1"
-AR Path="/604D6360/604F7C86" Ref="R7"  Part="1"
-F 0 "R7" V 10800 4900 50  0000 C CNN
+AR Path="/604D6360/604F7C86" Ref="R5"  Part="1"
+F 0 "R5" V 10800 4900 50  0000 C CNN
 F 1 "10K" V 11000 4900 50  0000 C CNN
 F 2 "Resistor_SMD:R_0805_2012Metric" H 10900 4900 50  0001 C CNN
@@
 P 4300 4450
 AR Path="/6057236E" Ref="C?"  Part="1"
-AR Path="/604D6360/6057236E" Ref="C8"  Part="1"
-F 0 "C8" H 4391 4496 50  0000 L CNN
+AR Path="/604D6360/6057236E" Ref="C7"  Part="1"
+F 0 "C7" H 4391 4496 50  0000 L CNN
 F 1 "0.1uF" H 4391 4405 50  0000 L CNN
 F 2 "Capacitor_SMD:C_0805_2012Metric" H 4300 4450 50  0001 C CNN
@@
 $EndComp
 $Comp
-L TI_TS3A4751PWR:TS3A4751PWR U?
-U 1 1 605723D0
-P 4950 4800
-AR Path="/605723D0" Ref="U?"  Part="1"
-AR Path="/604D6360/605723D0" Ref="U10"  Part="1"
-F 0 "U10" H 5550 5050 60  0000 C CNN
-F 1 "TS3A4751PWR" H 5550 4950 60  0000 C CNN
-F 2 "TI_TS3A4751PWR:TS3A4751PWR" H 6150 5040 60  0001 C CNN
-F 3 "" H 4950 4800 60  0000 C CNN
-	1    4950 4800
-	1    0    0    -1
-$EndComp
-$Comp
 L power:GNDD #PWR?
 U 1 1 605723D6
@@
 P 6150 4450
 AR Path="/6057242A" Ref="C?"  Part="1"
-AR Path="/604D6360/6057242A" Ref="C9"  Part="1"
-F 0 "C9" H 6241 4496 50  0000 L CNN
+AR Path="/604D6360/6057242A" Ref="C8"  Part="1"
+F 0 "C8" H 6241 4496 50  0000 L CNN
 F 1 "0.1uF" H 6241 4405 50  0000 L CNN
 F 2 "Capacitor_SMD:C_0805_2012Metric" H 6150 4450 50  0001 C CNN
@@
 $EndComp
 $Comp
-L Sensor_Magnetic:SM353LT U8
+L Sensor_Magnetic:SM353LT U9
 U 1 1 60643263
 P 1900 1600
-F 0 "U8" H 1570 1647 50  0000 R CNN
+F 0 "U9" H 1570 1647 50  0000 R CNN
 F 1 "SM353LT" H 1570 1554 50  0000 R CNN
 F 2 "Package_TO_SOT_SMD:SOT-23" H 1850 1600 50  0001 C CNN
@@
 DIGITAL LOGIC GROUND
 $Comp
-L Sensor_Magnetic:SM353LT U11
+L Sensor_Magnetic:SM353LT U10
 U 1 1 6065FC7B
 P 1900 2650
-F 0 "U11" H 1570 2697 50  0000 R CNN
+F 0 "U10" H 1570 2697 50  0000 R CNN
 F 1 "SM353LT" H 1570 2604 50  0000 R CNN
 F 2 "Package_TO_SOT_SMD:SOT-23" H 1850 2650 50  0001 C CNN
@@
 DIGITAL LOGIC GROUND
 $Comp
-L Sensor_Magnetic:SM353LT U12
+L Sensor_Magnetic:SM353LT U11
 U 1 1 60663056
 P 4250 1600
-F 0 "U12" H 3920 1647 50  0000 R CNN
+F 0 "U11" H 3920 1647 50  0000 R CNN
 F 1 "SM353LT" H 3920 1554 50  0000 R CNN
 F 2 "Package_TO_SOT_SMD:SOT-23" H 4200 1600 50  0001 C CNN
@@
 DIGITAL LOGIC GROUND
 $Comp
-L Sensor_Magnetic:SM353LT U13
+L Sensor_Magnetic:SM353LT U12
 U 1 1 606657C5
 P 4250 2650
-F 0 "U13" H 3920 2697 50  0000 R CNN
+F 0 "U12" H 3920 2697 50  0000 R CNN
 F 1 "SM353LT" H 3920 2604 50  0000 R CNN
 F 2 "Package_TO_SOT_SMD:SOT-23" H 4200 2650 50  0001 C CNN
@@
 Text Notes 750  850  0    100  ~ 0
 [ALTERNATE] HALL SWITCH ALTERNATES
-$Comp
-L TI_TS3A4751PWR:TS3A4751PWR U?
-U 1 1 60572422
-P 3100 4800
-AR Path="/60572422" Ref="U?"  Part="1"
-AR Path="/604D6360/60572422" Ref="U9"  Part="1"
-F 0 "U9" H 3650 5050 60  0000 C CNN
-F 1 "TS3A4751PWR" H 3650 4950 60  0000 C CNN
-F 2 "TI_TS3A4751PWR:TS3A4751PWR" H 4300 5040 60  0001 C CNN
-F 3 "" H 3100 4800 60  0000 C CNN
-	1    3100 4800
-	1    0    0    -1
-$EndComp
 Text Notes 7750 4400 0    50   ~ 0
 TOP MOUNTED
@@
 TOP MOUNTED
 $Comp
-L LiteOn_LTR-329ALS:LTR-329ALS-01 U14
+L LiteOn_LTR-329ALS:LTR-329ALS-01 U8
 U 1 1 603B38C5
 P 8250 6050
-F 0 "U14" H 8600 6350 60  0000 C CNN
+F 0 "U8" H 8600 6350 60  0000 C CNN
 F 1 "LTR-329ALS-01" H 9200 6350 60  0000 C CNN
 F 2 "LiteOn_LTR-329ALS:LTR-329ALS-01" H 9050 6290 60  0001 C CNN
@@
 	1    0    0    -1
 $EndComp
+$Comp
+L TI_TS3A4751PWR:TS3A4751PWR U?
+U 1 1 605723D0
+P 4950 4800
+AR Path="/605723D0" Ref="U?"  Part="1"
+AR Path="/604D6360/605723D0" Ref="U14"  Part="1"
+F 0 "U14" H 5550 5050 60  0000 C CNN
+F 1 "TS3A4751PWR" H 5550 4950 60  0000 C CNN
+F 2 "TI_TS3A4751PWR:TS3A4751PWR" H 6150 5040 60  0001 C CNN
+F 3 "" H 4950 4800 60  0000 C CNN
+	1    4950 4800
+	1    0    0    -1
+$EndComp
+$Comp
+L TI_TS3A4751PWR:TS3A4751PWR U?
+U 1 1 60572422
+P 3100 4800
+AR Path="/60572422" Ref="U?"  Part="1"
+AR Path="/604D6360/60572422" Ref="U13"  Part="1"
+F 0 "U13" H 3650 5050 60  0000 C CNN
+F 1 "TS3A4751PWR" H 3650 4950 60  0000 C CNN
+F 2 "TI_TS3A4751PWR:TS3A4751PWR" H 4300 5040 60  0001 C CNN
+F 3 "" H 3100 4800 60  0000 C CNN
+	1    3100 4800
+	1    0    0    -1
+$EndComp

Commit message: Core Board V0.6 remove bottom ALS, add new top ALS+PROX option
Parts:
- removed JP21, JP22, JP23, JP24: SolderJumper_2_Open, Jumper:SolderJumper-2_P1.3mm_Open_Pad1.0x1.5mm, symbol Jumper:SolderJumper_2_Open
- added JP17: SolderJumper_2_Open, Jumper:SolderJumper-2_P1.3mm_Open_Pad1.0x1.5mm, symbol Jumper:SolderJumper_2_Open
Connections:
- net ALS_INT: now also JP17.1 (A); no longer U6.2 (INT)
- net PLANE_5: now also U9.2 (OUTPUT)
- net PLANE_6: now also U10.2 (OUTPUT)
- net PLANE_7: now also U11.2 (OUTPUT)
- net PLANE_8: now also U12.2 (OUTPUT)
- new net: JP17.2 (B), U6.2 (INT)
Other:
- note removed: "TOP MOUNTED"
Changed lines of the file:
@@
 	7600 4900 6950 4900
 Wire Wire Line
-	6950 4900 6950 4500
-Text GLabel 7050 4500 2    50   Input ~ 0
+	6950 4900 6950 5600
+Text GLabel 7450 5600 2    50   Input ~ 0
 ALS_INT
 Wire Wire Line
-	6950 4500 7050 4500
+	6950 5600 7050 5600
 Text Notes 8600 4050 0    50   ~ 0
 SILKSCREEN: ALS I2C 0x29
@@
 Text Notes 9750 2700 0    50   ~ 0
 NOTE: These GPIO will be\nused by Core Plane Select\nif that option is enabled.
-$Comp
-L Jumper:SolderJumper_2_Open JP?
-U 1 1 6063DED0
-P 2450 1600
-AR Path="/6063DED0" Ref="JP?"  Part="1"
-AR Path="/604D6360/6063DED0" Ref="JP21"  Part="1"
-F 0 "JP21" H 2450 1700 50  0000 C CNN
-F 1 "SolderJumper_2_Open" H 2450 1720 50  0001 C CNN
-F 2 "Jumper:SolderJumper-2_P1.3mm_Open_Pad1.0x1.5mm" H 2450 1600 50  0001 C CNN
-F 3 "~" H 2450 1600 50  0001 C CNN
-	1    2450 1600
-	-1   0    0    -1
-$EndComp
-$Comp
-L Jumper:SolderJumper_2_Open JP?
-U 1 1 6063DED6
-P 2450 2650
-AR Path="/6063DED6" Ref="JP?"  Part="1"
-AR Path="/604D6360/6063DED6" Ref="JP22"  Part="1"
-F 0 "JP22" H 2450 2750 50  0000 C CNN
-F 1 "SolderJumper_2_Open" H 2450 2770 50  0001 C CNN
-F 2 "Jumper:SolderJumper-2_P1.3mm_Open_Pad1.0x1.5mm" H 2450 2650 50  0001 C CNN
-F 3 "~" H 2450 2650 50  0001 C CNN
-	1    2450 2650
-	-1   0    0    -1
-$EndComp
-$Comp
-L Jumper:SolderJumper_2_Open JP?
-U 1 1 6063DEE2
-P 4800 2650
-AR Path="/6063DEE2" Ref="JP?"  Part="1"
-AR Path="/604D6360/6063DEE2" Ref="JP24"  Part="1"
-F 0 "JP24" H 4800 2750 50  0000 C CNN
-F 1 "SolderJumper_2_Open" H 4800 2770 50  0001 C CNN
-F 2 "Jumper:SolderJumper-2_P1.3mm_Open_Pad1.0x1.5mm" H 4800 2650 50  0001 C CNN
-F 3 "~" H 4800 2650 50  0001 C CNN
-	1    4800 2650
-	-1   0    0    -1
-$EndComp
 Text GLabel 2600 1600 2    50   Output ~ 0
 PLANE_5
@@
 DIGITAL LOGIC GROUND
 $Comp
-L Jumper:SolderJumper_2_Open JP?
-U 1 1 6063DEDC
-P 4800 1600
-AR Path="/6063DEDC" Ref="JP?"  Part="1"
-AR Path="/604D6360/6063DEDC" Ref="JP23"  Part="1"
-F 0 "JP23" H 4800 1700 50  0000 C CNN
-F 1 "SolderJumper_2_Open" H 4800 1720 50  0001 C CNN
-F 2 "Jumper:SolderJumper-2_P1.3mm_Open_Pad1.0x1.5mm" H 4800 1600 50  0001 C CNN
-F 3 "~" H 4800 1600 50  0001 C CNN
-	1    4800 1600
-	-1   0    0    -1
-$EndComp
-$Comp
 L Sensor_Magnetic:SM353LT U9
 U 1 1 60643263
@@
 Text Notes 750  850  0    100  ~ 0
 [ALTERNATE] HALL SWITCH ALTERNATES
-Text Notes 7750 4400 0    50   ~ 0
-TOP MOUNTED
-Text Notes 9900 4400 0    50   ~ 0
-TOP MOUNTED
 $Comp
 L LiteOn_LTR-329ALS:LTR-329ALS-01 U8
@@
 Text Notes 8900 5550 0    50   ~ 0
 -OR-
-Text Notes 8750 5650 0    50   ~ 0
-TOP MOUNTED
 Text Notes 1800 1000 0    50   ~ 0
 To use Hall Switches, solder four SJs JP21-24.
@@
 	1    0    0    -1
 $EndComp
+Wire Wire Line
+	7350 5600 7450 5600
+$Comp
+L Jumper:SolderJumper_2_Open JP?
+U 1 1 617672C1
+P 7200 5600
+AR Path="/617672C1" Ref="JP?"  Part="1"
+AR Path="/604D6360/617672C1" Ref="JP17"  Part="1"
+F 0 "JP17" H 7200 5700 50  0000 C CNN
+F 1 "SolderJumper_2_Open" H 7200 5720 50  0001 C CNN
+F 2 "Jumper:SolderJumper-2_P1.3mm_Open_Pad1.0x1.5mm" H 7200 5600 50  0001 C CNN
+F 3 "~" H 7200 5600 50  0001 C CNN
+	1    7200 5600
+	-1   0    0    -1
+$EndComp
+Wire Wire Line
+	2300 1600 2600 1600
+Wire Wire Line
+	2300 2650 2600 2650
+Wire Wire Line
+	4650 2650 4950 2650
+Wire Wire Line
+	4650 1600 4950 1600
 $EndSCHEMATC

Commit message: CB V0.6 added ALS and PROX, removed bottom ALS, complete BOM, PNP, and Gerbers for fabrication
Parts:
- C7: renamed from C6; Description (none) -> Capacitor; Insert (none) -> YES; Value_Modifer (none) -> X7R ceramic
- C8: renamed from C7; Description (none) -> Capacitor; Insert (none) -> NO; Value_Modifer (none) -> X7R ceramic
- C9: renamed from C8; Description (none) -> Capacitor; Insert (none) -> NO; Value_Modifer (none) -> X7R ceramic
- JP1, JP10, JP11, JP12, JP13, JP14, JP15, JP16, JP17, JP2, JP3, JP4, JP5, JP6, JP7, JP8, JP9: Insert (none) -> NO
- R5: Description (none) -> Resistor; Insert (none) -> NO; Value_Modifer (none) -> 10%
- U10, U11, U12, U9: value SM353LT -> TCS40DPR,LF; Alt. Manufacturer (none) -> None; Alt. Mfg P/N (none) -> None; Description (none) -> Hall Switch (alternate); Insert (none) -> NO
- U13, U14: Description (none) -> Analog Switch Quad SPST (user-supplied optional); Insert (none) -> NO; Manufacturer_Name (none) -> TI; Mfg P/N (none) -> TS3A4751PWR
- U6: Alt. Manufacturer (none) -> None; Alt. Mfg P/N (none) -> None; Description (none) -> I2C Digital Light Sensor; Insert (none) -> NO; Manufacturer_Name (none) -> ROHM Semiconductor; Mfg P/N (none) -> BH1730FVC-TR
- U7: Alt. Manufacturer (none) -> None; Alt. Mfg P/N (none) -> None; Description (none) -> I2C Digital Light Sensor; Insert (none) -> NO; Manufacturer_Name (none) -> LiteOn; Mfg P/N (none) -> LTR-303ALS-01; Supplier (2nd) (none) -> Digi-Key; Supplier (Primary) (none) -> Mouser; Supplier SKU (2nd) (none) -> 160-2161-1-ND; Supplier SKU (Primary) (none) -> 859-LTR-303ALS-01
- U8: Alt. Manufacturer (none) -> None; Alt. Mfg P/N (none) -> None; Description (none) -> I2C Digital Light Sensor, DFN-4EP; Insert (none) -> YES; Manufacturer_Name (none) -> LiteOn; Mfg P/N (none) -> LTR-329ALS-01; Supplier (2nd) (none) -> Mouser; Supplier (Primary) (none) -> Arrow; Supplier SKU (2nd) (none) -> 859-LTR-329ALS-01; Supplier SKU (Primary) (none) -> LTR-329ALS-01; Value_Modifer (none) -> 4-DFN-EP (2x2)
- X1: Description (none) -> 2x6 Keyed Socket for SAO (user-supplied optional); Insert (none) -> NO
Other:
- note added: "A PLACE FOR AIR\nWIRES IF YOU WANT\nTO USE THE INTERRUPT"
- note added: "If Hall Switches are inserted, keep the decoupling caps on the first sheet.\nRecommended sensitivity ± (N and S) 3-7 mT (30-70 Gauss)\n(Toshiba TCS40DPR,LF is 4.4mT. Maybe Honeywell SM353LT ±2mT.)"
- note removed: "To use Hall Switches, solder four SJs JP21-24."
- moved on the sheet: U10, U11, U12, U9
